File: DapLink_STM32F103CBT6.kicad_sch (KiCad schematic)
At the start: 0 parts

Commit message: fabrication v1
Other:
- sheet Usb renamed UsbAndPower
- removed sheet Debug and UART Interface
- removed sheet MCU-LINK Power and USB
- sheet DebugAndUart ports: added TARGET_RESET, TARGET_RXD, TARGET_SWCLK, TARGET_SWDIO, TARGET_SWO, TARGET_TXD; removed none
- sheet Mcu ports: added TARGET_RESET, TARGET_RXD, TARGET_SWCLK, TARGET_SWDIO, TARGET_SWO, TARGET_TXD, USB_CONNECT, USB_D+, USB_D-; removed none
- sheet UsbAndPower: file Usb.kicad_sch -> UsbAndPower.kicad_sch
- sheet UsbAndPower ports: added USB_CONNECT, USB_D+, USB_D-; removed none
