File: DapLink_STM32F103CBT6.kicad_sch (KiCad schematic)
At the start: 0 parts

Commit message: add temp reference
Other:
- removed sheet Debug and UART Interface
- removed sheet MCU-LINK Power and USB
- added sheet LPC55S69-1 (Mcu.kicad_sch)
- added sheet LPC55S69-2 (Mcu.kicad_sch)
Changed lines of the file:
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@@
 	)
 	(sheet
-		(at 128.27 38.1)
-		(size 46.99 22.86)
+		(at 138.43 35.56)
+		(size 54.61 35.56)
 		(fields_autoplaced yes)
 		(stroke
@@
 			(color 0 0 0 0.0000)
 		)
-		(property "Sheetname" "Debug and UART Interface"
-			(at 128.27 37.3884 0)
+		(property "Sheetname" "LPC55S69-2"
+			(at 138.43 34.8484 0)
+			(show_name yes)
 			(effects
 				(font
@@
 			)
 		)
-		(property "Sheetfile" "mculink_standalone_debug_uart.kicad_sch"
-			(at 128.27 61.5446 0)
+		(property "Sheetfile" "Mcu.kicad_sch"
+			(at 138.43 71.7046 0)
 			(effects
 				(font
@@
 		)
 		(instances
-			(project "MCU-Link-Standalone"
-				(path "/52afa5f9-012e-424b-bf0c-786f4ecc122a"
+			(project "DapLink_STM32F103CBT6"
+				(path "/62d13f52-5b95-4b2e-9bc7-6f5f907932ec"
 					(page "3")
+				)
+			)
+		)
+	)
+	(sheet
+		(at 52.07 30.48)
+		(size 54.61 35.56)
+		(fields_autoplaced yes)
+		(stroke
+			(width 0.1524)
+			(type solid)
+		)
+		(fill
+			(color 0 0 0 0.0000)
+		)
+		(property "Sheetname" "LPC55S69-1"
+			(at 52.07 29.7684 0)
+			(show_name yes)
+			(effects
+				(font
+					(size 1.27 1.27)
+				)
+				(justify left bottom)
+			)
+		)
+		(property "Sheetfile" "Mcu.kicad_sch"
+			(at 52.07 66.6246 0)
+			(effects
+				(font
+					(size 1.27 1.27)
+				)
+				(justify left top)
+			)
+		)
+		(instances
+			(project "DapLink_STM32F103CBT6"
+				(path "/62d13f52-5b95-4b2e-9bc7-6f5f907932ec"
+					(page "2")
 				)
 			)
@@
 				)
 			)
-		)
-	)
-	(sheet
-		(at 71.12 38.1)
-		(size 48.26 22.86)
-		(fields_autoplaced yes)
-		(stroke
-			(width 0.1524)
-			(type solid)
-		)
-		(fill
-			(color 0 0 0 0.0000)
-		)
-		(property "Sheetname" "MCU-LINK Power and USB"
-			(at 71.12 37.3884 0)
-			(effects
-				(font
-					(size 1.27 1.27)
-				)
-				(justify left bottom)
-			)
-		)
-		(property "Sheetfile" "mculink_standalone_power_usb.kicad_sch"
-			(at 71.12 61.5446 0)
-			(effects
-				(font
-					(size 1.27 1.27)
-				)
-				(justify left top)
-			)
-		)
-		(instances
-			(project "MCU-Link-Standalone"
-				(path "/52afa5f9-012e-424b-bf0c-786f4ecc122a"
-					(page "2")
-				)
-			)

Commit message: TEMP
Other:
- removed sheet LPC55S69-1
- removed sheet LPC55S69-2
- added sheet Debug and UART Interface (mculink_standalone_debug_uart.kicad_sch)
- added sheet MCU-LINK Power and USB (mculink_standalone_power_usb.kicad_sch)
Changed lines of the file:
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@@
 	)
 	(sheet
-		(at 138.43 35.56)
-		(size 54.61 35.56)
+		(at 49.53 31.75)
+		(size 48.26 22.86)
 		(fields_autoplaced yes)
 		(stroke
@@
 			(color 0 0 0 0.0000)
 		)
-		(property "Sheetname" "LPC55S69-2"
-			(at 138.43 34.8484 0)
-			(show_name yes)
+		(property "Sheetname" "MCU-LINK Power and USB"
+			(at 49.53 31.0384 0)
 			(effects
 				(font
@@
 			)
 		)
-		(property "Sheetfile" "Mcu.kicad_sch"
-			(at 138.43 71.7046 0)
+		(property "Sheetfile" "mculink_standalone_power_usb.kicad_sch"
+			(at 49.53 55.1946 0)
+			(effects
+				(font
+					(size 1.27 1.27)
+				)
+				(justify left top)
+			)
+		)
+		(instances
+			(project "DapLink_STM32F103CBT6"
+				(path "/62d13f52-5b95-4b2e-9bc7-6f5f907932ec"
+					(page "2")
+				)
+			)
+		)
+	)
+	(sheet
+		(at 143.51 40.64)
+		(size 46.99 22.86)
+		(fields_autoplaced yes)
+		(stroke
+			(width 0.1524)
+			(type solid)
+		)
+		(fill
+			(color 0 0 0 0.0000)
+		)
+		(property "Sheetname" "Debug and UART Interface"
+			(at 143.51 39.9284 0)
+			(effects
+				(font
+					(size 1.27 1.27)
+				)
+				(justify left bottom)
+			)
+		)
+		(property "Sheetfile" "mculink_standalone_debug_uart.kicad_sch"
+			(at 143.51 64.0846 0)
 			(effects
 				(font
@@
 				)
 			)
-		)
-	)
-	(sheet
-		(at 52.07 30.48)
-		(size 54.61 35.56)
-		(fields_autoplaced yes)
-		(stroke
-			(width 0.1524)
-			(type solid)
-		)
-		(fill
-			(color 0 0 0 0.0000)
-		)
-		(property "Sheetname" "LPC55S69-1"
-			(at 52.07 29.7684 0)
-			(show_name yes)
-			(effects
-				(font
-					(size 1.27 1.27)
-				)
-				(justify left bottom)
-			)
-		)
-		(property "Sheetfile" "Mcu.kicad_sch"
-			(at 52.07 66.6246 0)
-			(effects
-				(font
-					(size 1.27 1.27)
-				)
-				(justify left top)
-			)
-		)
-		(instances
-			(project "DapLink_STM32F103CBT6"
-				(path "/62d13f52-5b95-4b2e-9bc7-6f5f907932ec"
-					(page "2")
-				)
-			)

Commit message: temp
Other:
- sheet Usb renamed UsbAndPower
- sheet UsbAndPower: file Usb.kicad_sch -> UsbAndPower.kicad_sch
Changed lines of the file:
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@@
 			(color 0 0 0 0.0000)
 		)
-		(property "Sheetname" "Usb"
+		(property "Sheetname" "UsbAndPower"
 			(at 156.21 91.9984 0)
 			(effects
@@
 			)
 		)
-		(property "Sheetfile" "Usb.kicad_sch"
+		(property "Sheetfile" "UsbAndPower.kicad_sch"
 			(at 156.21 119.9646 0)
 			(effects
@@
 			(project "DapLink_STM32F103CBT6"
 				(path "/62d13f52-5b95-4b2e-9bc7-6f5f907932ec"
-					(page "5")
+					(page "4")
 				)
 			)

Commit message: temp
Other:
- sheet DebugAndUart ports: added TARGET_RESET, TARGET_RXD, TARGET_SWCLK, TARGET_SWDIO, TARGET_SWO, TARGET_TXD; removed none
- sheet UsbAndPower ports: added USB_D+, USB_D-; removed none
Changed lines of the file:
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@@
+			)
+		)
+		(pin "USB_D-" bidirectional
+			(at 156.21 100.33 180)
+			(effects
+				(font
+					(size 1.27 1.27)
+				)
+				(justify left)
+			)
+		)
+		(pin "USB_D+" bidirectional
+			(at 156.21 104.14 180)
+			(effects
+				(font
+					(size 1.27 1.27)
+				)
+				(justify left)
 			)
 		)
@@
 			)
 		)
+		(pin "TARGET_TXD" output
+			(at 228.6 83.82 180)
+			(effects
+				(font
+					(size 1.27 1.27)
+				)
+				(justify left)
+			)
+		)
+		(pin "TARGET_RXD" input
+			(at 228.6 87.63 180)
+			(effects
+				(font
+					(size 1.27 1.27)
+				)
+				(justify left)
+			)
+		)
+		(pin "TARGET_SWO" output
+			(at 228.6 91.44 180)
+			(effects
+				(font
+					(size 1.27 1.27)
+				)
+				(justify left)
+			)
+		)
+		(pin "TARGET_RESET" output
+			(at 228.6 93.98 180)
+			(effects
+				(font
+					(size 1.27 1.27)
+				)
+				(justify left)
+			)
+		)
+		(pin "TARGET_SWDIO" bidirectional
+			(at 228.6 97.79 180)
+			(effects
+				(font
+					(size 1.27 1.27)
+				)
+				(justify left)
+			)
+		)
+		(pin "TARGET_SWCLK" output
+			(at 228.6 101.6 180)
+			(effects
+				(font
+					(size 1.27 1.27)
+				)
+				(justify left)
+			)
+		)

Commit message: temp
Other:
- sheet UsbAndPower ports: added USB_CONNECT; removed none
Changed lines of the file:
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@@
+			)
+		)
+		(pin "USB_CONNECT" input
+			(at 156.21 107.95 180)
+			(effects
+				(font
+					(size 1.27 1.27)
+				)
+				(justify left)
 			)
 		)

Commit message: temp
Changed lines of the file:
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@@
 	)
 	(sheet
-		(at 228.6 78.74)
-		(size 30.48 40.64)
+		(at 228.6 76.2)
+		(size 25.4 50.8)
 		(fields_autoplaced yes)
 		(stroke
@@
 		)
 		(property "Sheetname" "DebugAndUart"
-			(at 228.6 78.0284 0)
+			(at 228.6 75.4884 0)
 			(effects
 				(font
@@
 		)
 		(property "Sheetfile" "DebugAndUart.kicad_sch"
-			(at 228.6 119.9646 0)
+			(at 228.6 127.5846 0)
 			(effects
 				(font
@@
 			)
 		)
-		(pin "TARGET_TXD" output
-			(at 228.6 83.82 180)
+		(pin "TARGET_TXD" input
+			(at 228.6 88.9 180)
 			(effects
 				(font
@@
 			)
 		)
-		(pin "TARGET_RXD" input
-			(at 228.6 87.63 180)
-			(effects
-				(font
-					(size 1.27 1.27)
-				)
-				(justify left)
-			)
-		)
-		(pin "TARGET_SWO" output
+		(pin "TARGET_SWDIO" bidirectional
 			(at 228.6 91.44 180)
 			(effects
@@
 			)
 		)
-		(pin "TARGET_RESET" output
+		(pin "TARGET_RESET" input
 			(at 228.6 93.98 180)
 			(effects
@@
 			)
 		)
-		(pin "TARGET_SWDIO" bidirectional
-			(at 228.6 97.79 180)
+		(pin "TARGET_SWO" input
+			(at 228.6 96.52 180)
 			(effects
 				(font
@@
 			)
 		)
-		(pin "TARGET_SWCLK" output
+		(pin "TARGET_RXD" output
+			(at 228.6 99.06 180)
+			(effects
+				(font
+					(size 1.27 1.27)
+				)
+				(justify left)
+			)
+		)
+		(pin "TARGET_SWCLK" input
 			(at 228.6 101.6 180)
 			(effects

Commit message: temp
Other:
- removed sheet Debug and UART Interface
- removed sheet MCU-LINK Power and USB
Changed lines of the file:
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@@
-	)
-	(sheet
-		(at 49.53 31.75)
-		(size 48.26 22.86)
-		(fields_autoplaced yes)
-		(stroke
-			(width 0.1524)
-			(type solid)
-		)
-		(fill
-			(color 0 0 0 0.0000)
-		)
-		(property "Sheetname" "MCU-LINK Power and USB"
-			(at 49.53 31.0384 0)
-			(effects
-				(font
-					(size 1.27 1.27)
-				)
-				(justify left bottom)
-			)
-		)
-		(property "Sheetfile" "mculink_standalone_power_usb.kicad_sch"
-			(at 49.53 55.1946 0)
-			(effects
-				(font
-					(size 1.27 1.27)
-				)
-				(justify left top)
-			)
-		)
-		(instances
-			(project "DapLink_STM32F103CBT6"
-				(path "/62d13f52-5b95-4b2e-9bc7-6f5f907932ec"
-					(page "2")
-				)
-			)
-		)
-	)
-	(sheet
-		(at 143.51 40.64)
-		(size 46.99 22.86)
-		(fields_autoplaced yes)
-		(stroke
-			(width 0.1524)
-			(type solid)
-		)
-		(fill
-			(color 0 0 0 0.0000)
-		)
-		(property "Sheetname" "Debug and UART Interface"
-			(at 143.51 39.9284 0)
-			(effects
-				(font
-					(size 1.27 1.27)
-				)
-				(justify left bottom)
-			)
-		)
-		(property "Sheetfile" "mculink_standalone_debug_uart.kicad_sch"
-			(at 143.51 64.0846 0)
-			(effects
-				(font
-					(size 1.27 1.27)
-				)
-				(justify left top)
-			)
-		)
-		(instances
-			(project "DapLink_STM32F103CBT6"
-				(path "/62d13f52-5b95-4b2e-9bc7-6f5f907932ec"
-					(page "3")
-				)
-			)
-		)
 	)
 	(sheet
