File: DapLink_STM32F103CBT6.kicad_sch (KiCad schematic)
At the start: 0 parts

Commit message: temp
Other:
- sheet Mcu ports: added TARGET_RESET, TARGET_RXD, TARGET_SWCLK, TARGET_SWDIO, TARGET_SWO, TARGET_TXD, USB_CONNECT, USB_D+, USB_D-; removed none
Changed lines of the file:
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@@
 	)
 	(sheet
-		(at 156.21 92.71)
-		(size 40.64 26.67)
+		(at 80.01 90.17)
+		(size 24.13 22.86)
 		(fields_autoplaced yes)
 		(stroke
@@
 		)
 		(property "Sheetname" "UsbAndPower"
-			(at 156.21 91.9984 0)
+			(at 80.01 89.4584 0)
 			(effects
 				(font
@@
 		)
 		(property "Sheetfile" "UsbAndPower.kicad_sch"
-			(at 156.21 119.9646 0)
+			(at 80.01 113.6146 0)
 			(effects
 				(font
@@
 			)
 		)
+		(pin "USB_CONNECT" input
+			(at 104.14 104.14 0)
+			(effects
+				(font
+					(size 1.27 1.27)
+				)
+				(justify right)
+			)
+		)
+		(pin "USB_D+" bidirectional
+			(at 104.14 106.68 0)
+			(effects
+				(font
+					(size 1.27 1.27)
+				)
+				(justify right)
+			)
+		)
 		(pin "USB_D-" bidirectional
-			(at 156.21 100.33 180)
-			(effects
-				(font
-					(size 1.27 1.27)
-				)
-				(justify left)
-			)
-		)
-		(pin "USB_D+" bidirectional
-			(at 156.21 104.14 180)
-			(effects
-				(font
-					(size 1.27 1.27)
-				)
-				(justify left)
-			)
-		)
-		(pin "USB_CONNECT" input
-			(at 156.21 107.95 180)
-			(effects
-				(font
-					(size 1.27 1.27)
-				)
-				(justify left)
+			(at 104.14 109.22 0)
+			(effects
+				(font
+					(size 1.27 1.27)
+				)
+				(justify right)
 			)
 		)
@@
 	)
 	(sheet
-		(at 64.77 101.6)
-		(size 54.61 35.56)
+		(at 118.11 90.17)
+		(size 41.91 22.86)
 		(fields_autoplaced yes)
 		(stroke
@@
 		)
 		(property "Sheetname" "Mcu"
-			(at 64.77 100.8884 0)
+			(at 118.11 89.4584 0)
 			(effects
 				(font
@@
 		)
 		(property "Sheetfile" "Mcu.kicad_sch"
-			(at 64.77 137.7446 0)
+			(at 118.11 113.6146 0)
 			(effects
 				(font
@@
 				)
 				(justify left top)
+			)
+		)
+		(pin "TARGET_SWCLK" output
+			(at 160.02 99.06 0)
+			(effects
+				(font
+					(size 1.27 1.27)
+				)
+				(justify right)
+			)
+		)
+		(pin "TARGET_SWO" input
+			(at 160.02 96.52 0)
+			(effects
+				(font
+					(size 1.27 1.27)
+				)
+				(justify right)
+			)
+		)
+		(pin "TARGET_SWDIO" bidirectional
+			(at 160.02 101.6 0)
+			(effects
+				(font
+					(size 1.27 1.27)
+				)
+				(justify right)
+			)
+		)
+		(pin "USB_CONNECT" output
+			(at 118.11 104.14 180)
+			(effects
+				(font
+					(size 1.27 1.27)
+				)
+				(justify left)
+			)
+		)
+		(pin "TARGET_TXD" output
+			(at 160.02 104.14 0)
+			(effects
+				(font
+					(size 1.27 1.27)
+				)
+				(justify right)
+			)
+		)
+		(pin "TARGET_RXD" input
+			(at 160.02 106.68 0)
+			(effects
+				(font
+					(size 1.27 1.27)
+				)
+				(justify right)
+			)
+		)
+		(pin "USB_D-" bidirectional
+			(at 118.11 109.22 180)
+			(effects
+				(font
+					(size 1.27 1.27)
+				)
+				(justify left)
+			)
+		)
+		(pin "USB_D+" bidirectional
+			(at 118.11 106.68 180)
+			(effects
+				(font
+					(size 1.27 1.27)
+				)
+				(justify left)
+			)
+		)
+		(pin "TARGET_RESET" output
+			(at 160.02 109.22 0)
+			(effects
+				(font
+					(size 1.27 1.27)
+				)
+				(justify right)
 			)
 		)
@@
 	)
 	(sheet
-		(at 228.6 76.2)
-		(size 25.4 50.8)
+		(at 165.1 90.17)
+		(size 25.4 22.86)
 		(fields_autoplaced yes)
 		(stroke
@@
 		)
 		(property "Sheetname" "DebugAndUart"
-			(at 228.6 75.4884 0)
+			(at 165.1 89.4584 0)
 			(effects
 				(font
@@
 		)
 		(property "Sheetfile" "DebugAndUart.kicad_sch"
-			(at 228.6 127.5846 0)
+			(at 165.1 113.6146 0)
 			(effects
 				(font
@@
 		)
 		(pin "TARGET_TXD" input
-			(at 228.6 88.9 180)
+			(at 165.1 104.14 180)
 			(effects
 				(font
@@
 		)
 		(pin "TARGET_SWDIO" bidirectional
-			(at 228.6 91.44 180)
+			(at 165.1 101.6 180)
 			(effects
 				(font
@@
 		)
 		(pin "TARGET_RESET" input
-			(at 228.6 93.98 180)
+			(at 165.1 109.22 180)
 			(effects
 				(font
@@
 		)
 		(pin "TARGET_SWO" input
-			(at 228.6 96.52 180)
+			(at 165.1 96.52 180)
 			(effects
 				(font
@@
 		)
 		(pin "TARGET_RXD" output
-			(at 228.6 99.06 180)
+			(at 165.1 106.68 180)
 			(effects
 				(font
@@
 		)
 		(pin "TARGET_SWCLK" input
-			(at 228.6 101.6 180)
-			(effects
-				(font
+			(at 165.1 99.06 180)
+			(effects
+				(font

Commit message: temp
Changed lines of the file:
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@@
 		(company "roger225 Roger Jhang")
+	)
+	(wire
+		(pts
+			(xy 104.14 109.22) (xy 118.11 109.22)
+		)
+		(stroke
+			(width 0)
+			(type default)
+		)
+	)
+	(wire
+		(pts
+			(xy 160.02 99.06) (xy 165.1 99.06)
+		)
+		(stroke
+			(width 0)
+			(type default)
+		)
+	)
+	(wire
+		(pts
+			(xy 104.14 104.14) (xy 118.11 104.14)
+		)
+		(stroke
+			(width 0)
+			(type default)
+		)
+	)
+	(wire
+		(pts
+			(xy 160.02 101.6) (xy 165.1 101.6)
+		)
+		(stroke
+			(width 0)
+			(type default)
+		)
+	)
+	(wire
+		(pts
+			(xy 160.02 106.68) (xy 165.1 106.68)
+		)
+		(stroke
+			(width 0)
+			(type default)
+		)
+	)
+	(wire
+		(pts
+			(xy 104.14 106.68) (xy 118.11 106.68)
+		)
+		(stroke
+			(width 0)
+			(type default)
+		)
+	)
+	(wire
+		(pts
+			(xy 160.02 109.22) (xy 165.1 109.22)
+		)
+		(stroke
+			(width 0)
+			(type default)
+		)
+	)
+	(wire
+		(pts
+			(xy 160.02 104.14) (xy 165.1 104.14)
+		)
+		(stroke
+			(width 0)
+			(type default)
+		)
+	)
+	(wire
+		(pts
+			(xy 160.02 96.52) (xy 165.1 96.52)
+		)
+		(stroke
+			(width 0)
+			(type default)
+		)
 	)
 	(sheet
