File: DebugAndUart.kicad_sch (KiCad schematic)
At the start: 0 parts

Commit message: fabrication v1
Parts:
- added C22, C23: 0.1uF, Capacitor_SMD:C_0805_2012Metric, symbol Device:C
- added H1, H2, H3, H4: M3-3.2mm, MountingHole:MountingHole_3.2mm_M3_Pad_Via, symbol Mechanical:MountingHole_Pad
- added J5, J6: Conn_01x08_Pin, Connector_PinHeader_2.54mm:PinHeader_1x08_P2.54mm_Vertical, symbol Connector:Conn_01x08_Pin
- added Q5, Q6, Q7, Q8: SI2306, Package_TO_SOT_SMD:SOT-23, symbol Transistor_FET:ZXMN3A14F
- added R33, R39, R40, R44: 10K, Resistor_SMD:R_0805_2012Metric, symbol Device:R
- added R34, R35, R36: 100K, Resistor_SMD:R_0805_2012Metric, symbol Device:R
- added R37, R45: 4.7K, Resistor_SMD:R_0805_2012Metric, symbol Device:R
- added R38, R43: 100R, Resistor_SMD:R_0805_2012Metric, symbol Device:R
- added U6: TXB0104PW, Package_SO:TSSOP-14_4.4x5mm_P0.65mm, symbol Logic_LevelTranslator:TXB0104PW
Connections:
- new net: Q7.3 (D), Q8.1 (G), R44.1
- new net: Q5.1 (G), R38.1
- new net: R33.1, R34.2, U6.8 (OE)
- new net: Q7.1 (G), R43.1
- new net: Q5.3 (D), Q6.1 (G), R39.1
- new net +1.8V: C22.1, R33.2, R45.2, U6.1 (VCCA)
- new net +1.8V_Target: J6.1 (Pin_1)
- new net +3.3V: C23.1, J5.1 (Pin_1), R35.2, R39.2, R40.2, R44.2, U6.14 (VCCB)
- new net GND: C22.2, C23.2, H1.1, H2.1, H3.1, H4.1, J5.2 (Pin_2), J6.2 (Pin_2), Q5.2 (S), Q6.2 (S), Q7.2 (S), Q8.2 (S), R34.1, R36.1, R37.1, U6.7 (GND)
- new net TARGET_1v8_RESET: J6.8 (Pin_8), Q8.3 (D), R45.1
- new net TARGET_1v8_RXD: J6.6 (Pin_6), U6.2 (A1)
- new net TARGET_1v8_SWCLK: J6.3 (Pin_3), U6.5 (A4)
- new net TARGET_1v8_SWDIO: J6.4 (Pin_4), U6.4 (A3)
- new net TARGET_1v8_SWO: J6.7 (Pin_7), R37.2, R38.2
- new net TARGET_1v8_TXD: J6.5 (Pin_5), U6.3 (A2)
- new net TARGET_RESET: J5.8 (Pin_8), R43.2
- new net TARGET_RXD: J5.6 (Pin_6), U6.13 (B1)
- new net TARGET_SWCLK: J5.3 (Pin_3), R36.2, U6.10 (B4)
- new net TARGET_SWDIO: J5.4 (Pin_4), R35.1, U6.11 (B3)
- new net TARGET_SWO: J5.7 (Pin_7), Q6.3 (D), R40.1
- new net TARGET_TXD: J5.5 (Pin_5), U6.12 (B2)
