File: DebugAndUart.kicad_sch (KiCad schematic)
At the start: 0 parts

Commit message: temp
Parts:
- added J5, J6: Conn_01x06_Pin, Connector_PinHeader_2.54mm:PinHeader_1x06_P2.54mm_Vertical, symbol Connector:Conn_01x06_Pin
- added U8: TXB0104PW, Package_SO:TSSOP-14_4.4x5mm_P0.65mm, symbol Logic_LevelTranslator:TXB0104PW

Commit message: temp
Parts:
- removed J5, J6: Conn_01x06_Pin, Connector_PinHeader_2.54mm:PinHeader_1x06_P2.54mm_Vertical, symbol Connector:Conn_01x06_Pin
- added J5, J7: Conn_01x08_Pin, symbol Connector:Conn_01x08_Pin
Connections:
- net TARGET_RESET: now also J7.8 (Pin_8)
- net TARGET_RXD: now also J7.6 (Pin_6)
- net TARGET_SWCLK: now also J7.3 (Pin_3)
- net TARGET_SWDIO: now also J7.4 (Pin_4)
- net TARGET_SWO: now also J7.7 (Pin_7)
- net TARGET_TXD: now also J7.5 (Pin_5)
- new net TARGET_1v8_RESET: J5.8 (Pin_8)
- new net TARGET_1v8_RXD: J5.6 (Pin_6)
- new net TARGET_1v8_SWCLK: J5.3 (Pin_3)
- new net TARGET_1v8_SWDIO: J5.4 (Pin_4)
- new net TARGET_1v8_SWO: J5.7 (Pin_7)
- new net TARGET_1v8_TXD: J5.5 (Pin_5)
Changed lines of the file:
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@@
 		(company "roger225 Roger Jhang")
+	)
+	(label "TARGET_TXD"
+		(at 154.94 77.47 0)
+		(fields_autoplaced yes)
+		(effects
+			(font
+				(size 1.27 1.27)
+			)
+			(justify left bottom)
+		)
 	)
 	(label "TARGET_SWO"
@@
 		)
 	)
+	(label "TARGET_1v8_RESET"
+		(at 218.44 85.09 0)
+		(fields_autoplaced yes)
+		(effects
+			(font
+				(size 1.27 1.27)
+			)
+			(justify left bottom)
+		)
+	)
+	(label "TARGET_SWDIO"
+		(at 154.94 74.93 0)
+		(fields_autoplaced yes)
+		(effects
+			(font
+				(size 1.27 1.27)
+			)
+			(justify left bottom)
+		)
+	)
 	(label "TARGET_RXD"
 		(at 38.1 33.02 0)
@@
 		)
 	)
+	(label "TARGET_1v8_TXD"
+		(at 218.44 77.47 0)
+		(fields_autoplaced yes)
+		(effects
+			(font
+				(size 1.27 1.27)
+			)
+			(justify left bottom)
+		)
+	)
+	(label "TARGET_1v8_SWO"
+		(at 218.44 82.55 0)
+		(fields_autoplaced yes)
+		(effects
+			(font
+				(size 1.27 1.27)
+			)
+			(justify left bottom)
+		)
+	)
+	(label "TARGET_1v8_SWCLK"
+		(at 218.44 72.39 0)
+		(fields_autoplaced yes)
+		(effects
+			(font
+				(size 1.27 1.27)
+			)
+			(justify left bottom)
+		)
+	)
 	(label "TARGET_SWCLK"
 		(at 38.1 43.18 0)
@@
 		)
 	)
+	(label "TARGET_RXD"
+		(at 154.94 80.01 0)
+		(fields_autoplaced yes)
+		(effects
+			(font
+				(size 1.27 1.27)
+			)
+			(justify left bottom)
+		)
+	)
+	(label "TARGET_SWCLK"
+		(at 154.94 72.39 0)
+		(fields_autoplaced yes)
+		(effects
+			(font
+				(size 1.27 1.27)
+			)
+			(justify left bottom)
+		)
+	)
 	(label "TARGET_SWDIO"
 		(at 38.1 40.64 0)
@@
 		)
 	)
+	(label "TARGET_1v8_SWDIO"
+		(at 218.44 74.93 0)
+		(fields_autoplaced yes)
+		(effects
+			(font
+				(size 1.27 1.27)
+			)
+			(justify left bottom)
+		)
+	)
 	(label "TARGET_RESET"
 		(at 38.1 50.8 0)
@@
 		)
 	)
+	(label "TARGET_RESET"
+		(at 154.94 85.09 0)
+		(fields_autoplaced yes)
+		(effects
+			(font
+				(size 1.27 1.27)
+			)
+			(justify left bottom)
+		)
+	)
+	(label "TARGET_1v8_RXD"
+		(at 218.44 80.01 0)
+		(fields_autoplaced yes)
+		(effects
+			(font
+				(size 1.27 1.27)
+			)
+			(justify left bottom)
+		)
+	)
+	(label "TARGET_SWO"
+		(at 154.94 82.55 0)
+		(fields_autoplaced yes)
+		(effects
+			(font
+				(size 1.27 1.27)
+			)
+			(justify left bottom)
+		)
+	)
 	(symbol
-		(lib_id "Connector:Conn_01x06_Pin")
-		(at 149.86 72.39 0)
+		(lib_id "Connector:Conn_01x08_Pin")
+		(at 149.86 74.93 0)
 		(unit 1)
 		(exclude_from_sim no)
@@
 		(dnp no)
 		(fields_autoplaced yes)
-		(property "Reference" "J5"
+		(property "Reference" "J7"
 			(at 150.495 62.23 0)
 			(effects
@@
 			)
 		)
-		(property "Value" "Conn_01x06_Pin"
+		(property "Value" "Conn_01x08_Pin"
 			(at 150.495 64.77 0)
 			(effects
@@
 			)
 		)
-		(property "Footprint" "Connector_PinHeader_2.54mm:PinHeader_1x06_P2.54mm_Vertical"
-			(at 149.86 72.39 0)
+		(property "Footprint" ""
+			(at 149.86 74.93 0)
 			(effects
 				(font
@@
 		)
 		(property "Datasheet" "~"
-			(at 149.86 72.39 0)
-			(effects
-				(font
-					(size 1.27 1.27)
-				)
-				(hide yes)
-			)
-		)
-		(property "Description" "Generic connector, single row, 01x06, script generated"
-			(at 149.86 72.39 0)
-			(effects
-				(font
-					(size 1.27 1.27)
-				)
-				(hide yes)
-			)
+			(at 149.86 74.93 0)
+			(effects
+				(font
+					(size 1.27 1.27)
+				)
+				(hide yes)
+			)
+		)
+		(property "Description" "Generic connector, single row, 01x08, script generated"
+			(at 149.86 74.93 0)
+			(effects
+				(font
+					(size 1.27 1.27)
+				)
+				(hide yes)
+			)
+		)
+		(pin "8"
+		)
+		(pin "2"
+		)
+		(pin "1"
+		)
+		(pin "7"
+		)
+		(pin "4"
+		)
+		(pin "3"
+		)
+		(pin "6"
 		)
 		(pin "5"
-		)
-		(pin "1"
-		)
-		(pin "6"
-		)
-		(pin "4"
-		)
-		(pin "3"
-		)
-		(pin "2"
 		)
 		(instances
 			(project ""
 				(path "/62d13f52-5b95-4b2e-9bc7-6f5f907932ec/eb20876d-f6d4-40b4-9447-0949b56edc29"
-					(reference "J5")
+					(reference "J7")
 					(unit 1)
 				)
@@
 	)
 	(symbol
-		(lib_id "Connector:Conn_01x06_Pin")
-		(at 173.99 73.66 0)
+		(lib_id "Connector:Conn_01x08_Pin")
+		(at 213.36 74.93 0)
 		(unit 1)
 		(exclude_from_sim no)
@@
 		(dnp no)
 		(fields_autoplaced yes)
-		(property "Reference" "J6"
-			(at 174.625 63.5 0)
-			(effects
-				(font
-					(size 1.27 1.27)
-				)
-			)
-		)
-		(property "Value" "Conn_01x06_Pin"
-			(at 174.625 66.04 0)
-			(effects
-				(font
-					(size 1.27 1.27)
-				)
-			)
-		)
-		(property "Footprint" "Connector_PinHeader_2.54mm:PinHeader_1x06_P2.54mm_Vertical"
-			(at 173.99 73.66 0)
+		(property "Reference" "J5"
+			(at 213.995 62.23 0)
+			(effects
+				(font
+					(size 1.27 1.27)
+				)
+			)
+		)
+		(property "Value" "Conn_01x08_Pin"
+			(at 213.995 64.77 0)
+			(effects
+				(font
+					(size 1.27 1.27)
+				)
+			)
+		)
+		(property "Footprint" ""
+			(at 213.36 74.93 0)
 			(effects
 				(font
@@
 		)
 		(property "Datasheet" "~"
-			(at 173.99 73.66 0)
-			(effects
-				(font
-					(size 1.27 1.27)
-				)
-				(hide yes)
-			)
-		)
-		(property "Description" "Generic connector, single row, 01x06, script generated"
-			(at 173.99 73.66 0)
-			(effects
-				(font
-					(size 1.27 1.27)
-				)
-				(hide yes)
-			)
+			(at 213.36 74.93 0)
+			(effects
+				(font
+					(size 1.27 1.27)
+				)
+				(hide yes)
+			)
+		)
+		(property "Description" "Generic connector, single row, 01x08, script generated"
+			(at 213.36 74.93 0)
+			(effects
+				(font
+					(size 1.27 1.27)
+				)
+				(hide yes)
+			)
+		)
+		(pin "8"
+		)
+		(pin "2"
+		)
+		(pin "1"
+		)
+		(pin "7"
+		)
+		(pin "4"
+		)
+		(pin "3"
+		)
+		(pin "6"
 		)
 		(pin "5"
-		)
-		(pin "1"
-		)
-		(pin "6"
-		)
-		(pin "4"
-		)
-		(pin "3"
-		)
-		(pin "2"
 		)
 		(instances
 			(project "DapLink_STM32F103CBT6"
 				(path "/62d13f52-5b95-4b2e-9bc7-6f5f907932ec/eb20876d-f6d4-40b4-9447-0949b56edc29"
-					(reference "J6")
+					(reference "J5")
 					(unit 1)
 				)

Commit message: temp
Parts:
- added C38, C39: 0.1uF, Capacitor_SMD:C_0805_2012Metric, symbol Device:C
- added R12: 100K, Resistor_SMD:R_0805_2012Metric, symbol Device:R
- added R13: 10K, Resistor_SMD:R_0805_2012Metric, symbol Device:R
Connections:
- net TARGET_1v8_RXD: now also U8.5 (A4)
- net TARGET_1v8_SWCLK: now also U8.2 (A1)
- net TARGET_1v8_SWDIO: now also U8.3 (A2)
- net TARGET_1v8_TXD: now also U8.4 (A3)
- net TARGET_RXD: now also U8.10 (B4)
- net TARGET_SWCLK: now also U8.13 (B1)
- net TARGET_SWDIO: now also U8.12 (B2)
- net TARGET_TXD: now also U8.11 (B3)
- net +3.3V: now reaches J7.1 (Pin_1)
- net +3.3V: now also U8.14 (VCCB), C39.1
- net GND: now reaches J7.2 (Pin_2)
- net GND: now also J5.2 (Pin_2), U8.7 (GND), C38.2, C39.2, R12.1
- net +1.8V: now reaches J5.1 (Pin_1)
- net +1.8V: now also U8.1 (VCCA), C38.1, R13.2
- net at U8.8 (OE): now also R12.2, R13.1
Other:
- moved on the sheet: J5, J7, U8

Commit message: temp
Parts:
- added Q7: DMG2301L, Package_TO_SOT_SMD:SOT-23, symbol Transistor_FET:DMG2301L
- added R38: 100R, Resistor_SMD:R_0805_2012Metric, symbol Device:R
- added R39: 4.7k, Resistor_SMD:R_0805_2012Metric, symbol Device:R
- J5, J7: footprint (none) -> Connector_PinHeader_2.54mm:PinHeader_1x08_P2.54mm_Vertical
Connections:
- net +3.3V: now also Q7.2 (S)
- net GND: now also R39.1
- net TARGET_1v8_RESET: now also Q7.3 (D), R39.2
- net TARGET_RESET: now also R38.2
- new net: Q7.1 (G), R38.1
Other:
- moved on the sheet: J5

Commit message: temp
Parts:
- removed Q7: DMG2301L, Package_TO_SOT_SMD:SOT-23, symbol Transistor_FET:DMG2301L
- added Q6, Q7, Q8, Q9: SI2306, Package_TO_SOT_SMD:SOT-23, symbol Transistor_FET:ZXMN3A14F
- added R36, R37, R40: 10K, Resistor_SMD:R_0805_2012Metric, symbol Device:R
- added R41, R42: 4.7K, Resistor_SMD:R_0805_2012Metric, symbol Device:R
- R39: value 4.7k -> 100R
Connections:
- net +1.8V: now also R41.2
- net +3.3V: now also R36.2, R37.2, R40.2
- net GND: now also Q6.2 (S), Q7.2 (S), Q8.2 (S), Q9.2 (S), R42.1; no longer R39.1
- net TARGET_1v8_RESET: now also Q7.3 (D), R41.1; no longer R39.2
- net TARGET_1v8_SWO: now also R39.2, R42.2
- net TARGET_SWO: now also Q9.3 (D), R40.1
- net at R38.1: now also Q6.1 (G)
- new net: Q6.3 (D), Q7.1 (G), R36.1
- new net: Q8.1 (G), R39.1
- new net: Q8.3 (D), Q9.1 (G), R37.1
Other:
- moved on the sheet: J5, J7, R12, R38

Commit message: temp
Parts:
- added R34, R35: 100K, Resistor_SMD:R_0805_2012Metric, symbol Device:R
Connections:
- net +3.3V: now also R34.2
- net GND: now also R35.1
- net TARGET_SWCLK: now also R35.2
- net TARGET_SWDIO: now also R34.1

Commit message: temp
Parts:
- added H7: RXD, mculink:castellated pin, symbol Mechanical:MountingHole_Pad
Changed lines of the file:
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@@
+	)
+	(symbol
+		(lib_id "Mechanical:MountingHole_Pad")
+		(at 48.26 121.92 0)
+		(unit 1)
+		(exclude_from_sim no)
+		(in_bom no)
+		(on_board yes)
+		(dnp no)
+		(property "Reference" "H7"
+			(at 46.99 115.57 0)
+			(effects
+				(font
+					(size 1.27 1.27)
+				)
+				(justify left)
+				(hide yes)
+			)
+		)
+		(property "Value" "RXD"
+			(at 46.99 118.11 0)
+			(effects
+				(font
+					(size 1.27 1.27)
+				)
+				(justify left)
+			)
+		)
+		(property "Footprint" "mculink:castellated pin"
+			(at 48.26 121.92 0)
+			(effects
+				(font
+					(size 1.27 1.27)
+				)
+				(hide yes)
+			)
+		)
+		(property "Datasheet" "~"
+			(at 48.26 121.92 0)
+			(effects
+				(font
+					(size 1.27 1.27)
+				)
+				(hide yes)
+			)
+		)
+		(property "Description" ""
+			(at 48.26 121.92 0)
+			(effects
+				(font
+					(size 1.27 1.27)
+				)
+				(hide yes)
+			)
+		)
+		(pin "1"
+		)
+		(instances
+			(project "DapLink_STM32F103CBT6"
+				(path "/62d13f52-5b95-4b2e-9bc7-6f5f907932ec/eb20876d-f6d4-40b4-9447-0949b56edc29"
+					(reference "H7")
+					(unit 1)
+				)
+			)
+		)
 	)
 	(symbol
