File: DebugAndUart.kicad_sch (KiCad schematic)
At the start: 21 parts, among them J5 Conn_01x08_Pin, J7 Conn_01x08_Pin, Q6 SI2306, Q7 SI2306, Q8 SI2306, Q9 SI2306, U8 TXB0104PW

Commit message: temp
Parts:
- added R7, R8: 0R, Resistor_SMD:R_0805_2012Metric, symbol Device:R
Connections:
- net +1.8V: now also R7.1, R8.2; no longer J5.1 (Pin_1)
- new net +1.8V_LDO: R7.2
- new net +1.8V_Target: J5.1 (Pin_1), R8.1

Commit message: temp
Parts:
- renumbered C38 to C22, C39 to C23, H7 to H1, J7 to J5, J5 to J6, Q8 to Q5, Q9 to Q6, Q6 to Q7, Q7 to Q8, R13 to R33, R12 to R34, R34 to R35, R35 to R36, R42 to R37, R39 to R38, R37 to R39, R7 to R41, R8 to R42, R38 to R43, R36 to R44, R41 to R45, U8 to U6

Commit message: temp
Parts:
- added H2, H3, H4: M3-3.2mm, MountingHole:MountingHole_3.2mm_M3_Pad_Via, symbol Mechanical:MountingHole_Pad
- added J7: Conn_01x03_Pin, Connector_PinHeader_2.54mm:PinHeader_1x03_P2.54mm_Vertical, symbol Connector:Conn_01x03_Pin
- H1: value RXD -> M3-3.2mm; footprint mculink:castellated pin -> MountingHole:MountingHole_3.2mm_M3_Pad_Via
Connections:
- net +1.8V: now also J7.2 (Pin_2)
- net +1.8V_LDO: now also J7.3 (Pin_3)
- net +1.8V_Target: now also J7.1 (Pin_1)
- net GND: now also H1.1, H2.1, H3.1, H4.1

Commit message: temp
Parts:
- removed J7: Conn_01x03_Pin, Connector_PinHeader_2.54mm:PinHeader_1x03_P2.54mm_Vertical, symbol Connector:Conn_01x03_Pin
- removed R41, R42: 0R, Resistor_SMD:R_0805_2012Metric, symbol Device:R

Commit message: temp
Connections:
- net TARGET_1v8_RXD: now also U6.2 (A1); no longer U6.5 (A4)
- net TARGET_1v8_SWCLK: now also U6.5 (A4); no longer U6.2 (A1)
- net TARGET_1v8_SWDIO: now also U6.4 (A3); no longer U6.3 (A2)
- net TARGET_1v8_TXD: now also U6.3 (A2); no longer U6.4 (A3)
- net TARGET_RXD: now also U6.13 (B1); no longer U6.10 (B4)
- net TARGET_SWCLK: now also U6.10 (B4); no longer U6.13 (B1)
- net TARGET_SWDIO: now also U6.11 (B3); no longer U6.12 (B2)
- net TARGET_TXD: now also U6.12 (B2); no longer U6.11 (B3)
Other:
- moved on the sheet: R35, R36

Commit message: temp
Other:
- moved on the sheet: R35, R36
Changed lines of the file:
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@@
 	(wire
 		(pts
-			(xy 100.33 62.23) (xy 100.33 64.77)
+			(xy 104.14 62.23) (xy 104.14 64.77)
 		)
 		(stroke
@@
 	(wire
 		(pts
-			(xy 100.33 78.74) (xy 100.33 80.01)
+			(xy 104.14 78.74) (xy 104.14 80.01)
 		)
 		(stroke
@@
 	(wire
 		(pts
-			(xy 100.33 53.34) (xy 100.33 54.61)
+			(xy 104.14 53.34) (xy 104.14 54.61)
 		)
 		(stroke
@@
 	(wire
 		(pts
-			(xy 82.55 64.77) (xy 100.33 64.77)
+			(xy 82.55 64.77) (xy 104.14 64.77)
 		)
 		(stroke
@@
 	(wire
 		(pts
-			(xy 100.33 69.85) (xy 100.33 71.12)
+			(xy 104.14 69.85) (xy 104.14 71.12)
 		)
 		(stroke
@@
 	(wire
 		(pts
-			(xy 82.55 69.85) (xy 100.33 69.85)
+			(xy 82.55 69.85) (xy 104.14 69.85)
 		)
 		(stroke
@@
 	(symbol
 		(lib_id "Device:R")
-		(at 100.33 58.42 180)
+		(at 104.14 58.42 180)
 		(unit 1)
 		(exclude_from_sim no)
@@
 		(fields_autoplaced yes)
 		(property "Reference" "R35"
-			(at 102.87 57.1499 0)
+			(at 106.68 57.1499 0)
 			(effects
 				(font
@@
 		)
 		(property "Value" "100K"
-			(at 102.87 59.6899 0)
+			(at 106.68 59.6899 0)
 			(effects
 				(font
@@
 		)
 		(property "Footprint" "Resistor_SMD:R_0805_2012Metric"
-			(at 102.108 58.42 90)
+			(at 105.918 58.42 90)
 			(effects
 				(font
@@
 		)
 		(property "Datasheet" "~"
-			(at 100.33 58.42 0)
+			(at 104.14 58.42 0)
 			(effects
 				(font
@@
 		)
 		(property "Description" "Resistor"
-			(at 100.33 58.42 0)
+			(at 104.14 58.42 0)
 			(effects
 				(font
@@
 	(symbol
 		(lib_id "power:+3.3V")
-		(at 100.33 53.34 0)
+		(at 104.14 53.34 0)
 		(unit 1)
 		(exclude_from_sim no)
@@
 		(fields_autoplaced yes)
 		(property "Reference" "#PWR050"
-			(at 100.33 57.15 0)
+			(at 104.14 57.15 0)
 			(effects
 				(font
@@
 		)
 		(property "Value" "+3.3V"
-			(at 100.33 48.26 0)
+			(at 104.14 48.26 0)
 			(effects
 				(font
@@
 		)
 		(property "Footprint" ""
-			(at 100.33 53.34 0)
+			(at 104.14 53.34 0)
 			(effects
 				(font
@@
 		)
 		(property "Datasheet" ""
-			(at 100.33 53.34 0)
+			(at 104.14 53.34 0)
 			(effects
 				(font
@@
 		)
 		(property "Description" "Power symbol creates a global label with name \"+3.3V\""
-			(at 100.33 53.34 0)
+			(at 104.14 53.34 0)
 			(effects
 				(font
@@
 	(symbol
 		(lib_id "power:GND")
-		(at 100.33 80.01 0)
+		(at 104.14 80.01 0)
 		(unit 1)
 		(exclude_from_sim no)
@@
 		(fields_autoplaced yes)
 		(property "Reference" "#PWR051"
-			(at 100.33 86.36 0)
+			(at 104.14 86.36 0)
 			(effects
 				(font
@@
 		)
 		(property "Value" "GND"
-			(at 100.33 85.09 0)
+			(at 104.14 85.09 0)
 			(effects
 				(font
@@
 		)
 		(property "Footprint" ""
-			(at 100.33 80.01 0)
+			(at 104.14 80.01 0)
 			(effects
 				(font
@@
 		)
 		(property "Datasheet" ""
-			(at 100.33 80.01 0)
+			(at 104.14 80.01 0)
 			(effects
 				(font
@@
 		)
 		(property "Description" "Power symbol creates a global label with name \"GND\" , ground"
-			(at 100.33 80.01 0)
+			(at 104.14 80.01 0)
 			(effects
 				(font
@@
 	(symbol
 		(lib_id "Device:R")
-		(at 100.33 74.93 180)
+		(at 104.14 74.93 180)
 		(unit 1)
 		(exclude_from_sim no)
@@
 		(fields_autoplaced yes)
 		(property "Reference" "R36"
-			(at 102.87 73.6599 0)
+			(at 106.68 73.6599 0)
 			(effects
 				(font
@@
 		)
 		(property "Value" "100K"
-			(at 102.87 76.1999 0)
+			(at 106.68 76.1999 0)
 			(effects
 				(font
@@
 		)
 		(property "Footprint" "Resistor_SMD:R_0805_2012Metric"
-			(at 102.108 74.93 90)
+			(at 105.918 74.93 90)
 			(effects
 				(font
@@
 		)
 		(property "Datasheet" "~"
-			(at 100.33 74.93 0)
+			(at 104.14 74.93 0)
 			(effects
 				(font
@@
 		)
 		(property "Description" "Resistor"
-			(at 100.33 74.93 0)
+			(at 104.14 74.93 0)
 			(effects
 				(font
