File: Mcu.kicad_sch (KiCad schematic)
At the start: 0 parts

Commit message: fabrication v1
Parts:
- added C1, C10, C5, C7, C8, C9: 0.1uF, Capacitor_SMD:C_0805_2012Metric, symbol Device:C
- added C2, C3: 22pF, Capacitor_SMD:C_0603_1608Metric, symbol Device:C
- added C6: 1uF 10V X7R, Capacitor_SMD:C_1206_3216Metric, symbol Device:C
- added D1: HID, LED_SMD:LED_0805_2012Metric, symbol Device:LED
- added D2: CDC, LED_SMD:LED_0805_2012Metric, symbol Device:LED
- added D3: MSC, LED_SMD:LED_0805_2012Metric, symbol Device:LED
- added D4: CONNECTED, LED_SMD:LED_0805_2012Metric, symbol Device:LED
- added D5: RUNNING, LED_SMD:LED_0805_2012Metric, symbol Device:LED
- added D6: TX, LED_SMD:LED_0805_2012Metric, symbol Device:LED
- added D7: RX, LED_SMD:LED_0805_2012Metric, symbol Device:LED
- added J1, J2: Conn_01x03_Pin, Connector_PinHeader_2.54mm:PinHeader_1x03_P2.54mm_Vertical, symbol Connector:Conn_01x03_Pin
- added J3: Conn_01x08_Pin, Connector_PinHeader_2.54mm:PinHeader_1x08_P2.54mm_Vertical, symbol Connector:Conn_01x08_Pin
- added Q1, Q2: SI2306, Package_TO_SOT_SMD:SOT-23, symbol Transistor_FET:ZXMN3A14F
- added R1, R2, R3: 1.5k, Resistor_SMD:R_0805_2012Metric, symbol Device:R
- added R10, R11, R14, R15, R16, R17, R8: 22R, Resistor_SMD:R_0805_2012Metric, symbol Device:R
- added R12, R13: 100R, Resistor_SMD:R_0805_2012Metric, symbol Device:R
- added R18, R19: 4.7K, Resistor_SMD:R_0805_2012Metric, symbol Device:R
- added R20, R23: 100, Resistor_SMD:R_0805_2012Metric, symbol Device:R
- added R21, R4: 10K, Resistor_SMD:R_0805_2012Metric, symbol Device:R
- added R22, R24, R5, R6: 470R, Resistor_SMD:R_0805_2012Metric, symbol Device:R
- added R7, R9: 10k, Resistor_SMD:R_0805_2012Metric, symbol Device:R
- added SW1: SKQGAFE010, Button_Switch_SMD:SW_SPST_SKQG_WithStem, symbol Switch:SW_Push
- added U1: STM32F103CBTx, Package_QFP:LQFP-48_7x7mm_P0.5mm, symbol MCU_ST_STM32F1:STM32F103CBTx
- added Y1: Crystal_GND24, Crystal:Crystal_SMD_3225-4Pin_3.2x2.5mm, symbol Device:Crystal_GND24
Connections:
- new net: Q1.1 (G), R20.2
- new net: D6.1 (K), Q1.3 (D)
- new net: D1.1 (K), R1.2
- new net: D3.1 (K), R3.2
- new net: Q2.1 (G), R23.2
- new net: D6.2 (A), R22.2
- new net: R9.1, U1.20 (PB2)
- new net: R10.1, U1.26 (PB13)
- new net: D5.2 (A), R6.1
- new net: R15.2, U1.13 (PA3)
- new net: R14.2, U1.12 (PA2)
- new net: R12.1, U1.25 (PB12)
- new net: R11.1, R12.2, U1.27 (PB14)
- new net: R18.1, R19.2, U1.10 (PA0)
- new net: R8.1, U1.18 (PB0)
- new net: R13.1, U1.28 (PB15)
- new net: R16.2, U1.32 (PA11)
- new net: R17.2, U1.33 (PA12)
- new net: R7.1, U1.44 (BOOT0)
- new net: D4.2 (A), R5.1
- new net: D7.2 (A), R24.2
- new net: D7.1 (K), Q2.3 (D)
- new net: D2.1 (K), R2.2
- new net +3.3V: C5.1, C6.1, C7.1, C8.1, C9.1, D1.2 (A), D2.2 (A), D3.2 (A), J1.1 (Pin_1), J2.1 (Pin_1), J3.1 (Pin_1), R18.2, R21.2, R22.1, R24.1, R4.2, U1.1 (VBAT), U1.24 (VDD), U1.36 (VDD), U1.48 (VDD), U1.9 (VDDA)
- new net BOOT0: J2.2 (Pin_2), R7.2
- new net BOOT1: J1.2 (Pin_2), R9.2
- new net GND: C1.2, C10.2, C2.1, C3.2, C5.2, C6.2, C7.2, C8.2, C9.2, D4.1 (K), D5.1 (K), J1.3 (Pin_3), J2.3 (Pin_3), J3.2 (Pin_2), Q1.2 (S), Q2.2 (S), R19.1, SW1.1, U1.23 (VSS), U1.35 (VSS), U1.47 (VSS), U1.8 (VSSA), Y1.2, Y1.4
- new net IF_RESET: C10.1, J3.8 (Pin_8), R21.1, U1.7 (NRST)
- new net IF_RXD: J3.6 (Pin_6), R23.1, U1.31 (PA10)
- new net IF_SWCLK: J3.3 (Pin_3), U1.37 (PA14)
- new net IF_SWDIO: J3.4 (Pin_4), U1.34 (PA13)
- new net IF_SWO: J3.7 (Pin_7), U1.39 (PB3)
- new net IF_TXD: J3.5 (Pin_5), R20.1, U1.30 (PA9)
- new net LED_CONNECTED: R5.2, U1.42 (PB6)
- new net LED_RUNNING: R6.2, U1.29 (PA8)
- new net LED_nCDC: R2.1, U1.16 (PA6)
- new net LED_nHID: R1.1, U1.15 (PA5)
- new net LED_nMSC: R3.1, U1.17 (PA7)
- new net OSC_IN: C2.2, U1.5 (PD0), Y1.3
- new net OSC_OUT: C3.1, U1.6 (PD1), Y1.1
- new net TARGET_RESET: C1.1, R4.1, R8.2, SW1.2
- new net TARGET_RXD: R15.1
- new net TARGET_SWCLK: R10.2
- new net TARGET_SWDIO: R11.2
- new net TARGET_SWO: R13.2
- new net TARGET_TXD: R14.1
- new net USB_CONNECT: U1.38 (PA15)
- new net USB_D+: R17.1
- new net USB_D-: R16.1
