File: Mcu.kicad_sch (KiCad schematic)
At the start: 26 parts, among them J2 BM03B-SRSS-TB, J3 Conn_02x05_Odd_Even, Q1 PMDXB290UNE, Q2 PMDXB290UNE, Q3 PMDXB290UNE, SW1 KMR221GLFS, U2 LPC55S69JBD64, U3 STMPS2141STR

Commit message: TEMP
Parts:
- removed D2, D5: PESD5V0L5UV, Package_TO_SOT_SMD:SOT-666, symbol Power_Protection:PESD5V0L5UV
- removed D3: LED_RED, LED_SMD:LED_0402_1005Metric, symbol Device:LED
- removed D4: PMEG3005AESFYL, Diode_SMD:Nexperia_DSN0603-2_0.6x0.3mm_P0.4mm, symbol Device:D_Schottky
- removed H10: Reset, mculink:castellated pin, symbol Mechanical:MountingHole_Pad
- removed H5: RXD, mculink:castellated pin, symbol Mechanical:MountingHole_Pad
- removed H6: SWCLK, mculink:castellated pin, symbol Mechanical:MountingHole_Pad
- removed H7: TXD, mculink:castellated pin, symbol Mechanical:MountingHole_Pad
- removed H8: SWDIO, mculink:castellated pin, symbol Mechanical:MountingHole_Pad
- removed H9: 3.3V, mculink:castellated pin, symbol Mechanical:MountingHole_Pad
- removed J2: BM03B-SRSS-TB, mculink:JST_BM03B-SRSS-TB_LF__SN_, symbol mculink:BM03B-SRSS-TB_LF__SN_
- removed J3: Conn_02x05_Odd_Even, mculink:SWD_Pin_Header_Straight_2x05_Pitch1.27mm_SMD, symbol Connector_Generic:Conn_02x05_Odd_Even
- removed JP1: SWD disable, Jumper:SolderJumper-2_P1.3mm_Open_RoundedPad1.0x1.5mm, symbol Jumper:Jumper_2_Bridged
- removed Q1, Q2, Q3: PMDXB290UNE, mculink:SOT1216, symbol Transistor_FET:FDG6335N
- removed R10, R6: 2k, Resistor_SMD:R_0402_1005Metric, symbol Device:R
- removed R11: 10, Resistor_SMD:R_0402_1005Metric, symbol Device:R
- removed R5: 10k, Resistor_SMD:R_0402_1005Metric, symbol Device:R
- removed R7: 100, Resistor_SMD:R_0402_1005Metric, symbol Device:R
- removed R8, R9: 100k, Resistor_SMD:R_0402_1005Metric, symbol Device:R
- removed SW1: KMR221GLFS, mculink:SW_C_K_KMR2, symbol mculink_kicad:KMR221GLFS
- removed U2: LPC55S69JBD64, mculink:LQFP-64-1EP_10x10mm_P0.5mm_EP5x5mm, symbol mculink_kicad:LPC55S69JBD64
- removed U3: STMPS2141STR, mculink:SOT95P280X145-5N, symbol mculink:STMPS2141STR
Connections:
- no-connect marks 28 -> 0
Other:
- note removed: "Connect to GND: Disable second VCOM"
- note removed: "Cortex Debug (SWD/JTAG) interface"
- note removed: "Current Protection"
- note removed: "Enable ISP mode"
- note removed: "LED: SWD activity"
- note removed: "Open: Boot from internal FLASH Closed: Enable ISP mode (USB or UART)"
- note removed: "SWDIO/TMS SWCLK/TCK SWO/TDO -/TDI RESET"
- note removed: "Signal isolation"
- note removed: "UART Interface to Target"
- note removed: "VREF GND GND ISP-EN GND (detect)"
- note removed: "castellated pins"
- note removed: "eFuse and Reverse"
- note removed: "when switched off"
