File: Mcu.kicad_sch (KiCad schematic)
At the start: 0 parts

Commit message: temp
Parts:
- added U9: STM32F103CBTx, Package_QFP:LQFP-48_7x7mm_P0.5mm, symbol MCU_ST_STM32F1:STM32F103CBTx
Connections:
- new net: U9.23 (VSS), U9.35 (VSS), U9.47 (VSS)
Changed lines of the file:
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@@
 		(company "roger225 Roger Jhang")
 	)
+	(symbol
+		(lib_id "MCU_ST_STM32F1:STM32F103CBTx")
+		(at 140.97 100.33 0)
+		(unit 1)
+		(exclude_from_sim no)
+		(in_bom yes)
+		(on_board yes)
+		(dnp no)
+		(fields_autoplaced yes)
+		(property "Reference" "U9"
+			(at 145.7041 138.43 0)
+			(effects
+				(font
+					(size 1.27 1.27)
+				)
+				(justify left)
+			)
+		)
+		(property "Value" "STM32F103CBTx"
+			(at 145.7041 140.97 0)
+			(effects
+				(font
+					(size 1.27 1.27)
+				)
+				(justify left)
+			)
+		)
+		(property "Footprint" "Package_QFP:LQFP-48_7x7mm_P0.5mm"
+			(at 128.27 135.89 0)
+			(effects
+				(font
+					(size 1.27 1.27)
+				)
+				(justify right)
+				(hide yes)
+			)
+		)
+		(property "Datasheet" "https://www.st.com/resource/en/datasheet/stm32f103cb.pdf"
+			(at 140.97 100.33 0)
+			(effects
+				(font
+					(size 1.27 1.27)
+				)
+				(hide yes)
+			)
+		)
+		(property "Description" "STMicroelectronics Arm Cortex-M3 MCU, 128KB flash, 20KB RAM, 72 MHz, 2.0-3.6V, 37 GPIO, LQFP48"
+			(at 140.97 100.33 0)
+			(effects
+				(font
+					(size 1.27 1.27)
+				)
+				(hide yes)
+			)
+		)
+		(pin "24"
+		)
+		(pin "3"
+		)
+		(pin "10"
+		)
+		(pin "13"
+		)
+		(pin "19"
+		)
+		(pin "33"
+		)
+		(pin "34"
+		)
+		(pin "26"
+		)
+		(pin "9"
+		)
+		(pin "25"
+		)
+		(pin "40"
+		)
+		(pin "44"
+		)
+		(pin "8"
+		)
+		(pin "23"
+		)
+		(pin "39"
+		)
+		(pin "11"
+		)
+		(pin "18"
+		)
+		(pin "12"
+		)
+		(pin "28"
+		)
+		(pin "31"
+		)
+		(pin "41"
+		)
+		(pin "4"
+		)
+		(pin "45"
+		)
+		(pin "21"
+		)
+		(pin "17"
+		)
+		(pin "27"
+		)
+		(pin "29"
+		)
+		(pin "43"
+		)
+		(pin "47"
+		)
+		(pin "6"
+		)
+		(pin "7"
+		)
+		(pin "14"
+		)
+		(pin "2"
+		)
+		(pin "16"
+		)
+		(pin "35"
+		)
+		(pin "36"
+		)
+		(pin "37"
+		)
+		(pin "20"
+		)
+		(pin "42"
+		)
+		(pin "48"
+		)
+		(pin "38"
+		)
+		(pin "1"
+		)
+		(pin "5"
+		)
+		(pin "15"
+		)
+		(pin "30"
+		)
+		(pin "32"
+		)
+		(pin "46"
+		)
+		(pin "22"
+		)
+		(instances
+			(project ""
+				(path "/62d13f52-5b95-4b2e-9bc7-6f5f907932ec/c5505282-deed-4b2e-81f9-216594ebbe5e"
+					(reference "U9")
+					(unit 1)
+				)
+			)
+		)
+	)
 )

Commit message: temp
Parts:
- added C40, C41, C42, C43, C44, C46: 0.1uF, Capacitor_SMD:C_0805_2012Metric, symbol Device:C
- added C45: 1uF 10V X7R, Capacitor_SMD:C_1206_3216Metric, symbol Device:C
- added J6: Conn_01x08_Pin, symbol Connector:Conn_01x08_Pin
- added R14, R25: 10K, Resistor_SMD:R_0805_2012Metric, symbol Device:R
- added R23, R24: 100R, Resistor_SMD:R_0805_2012Metric, symbol Device:R
- added SW2: SW_Push, Button_Switch_SMD:SW_SPST_B3S-1000, symbol Switch:SW_Push
Connections:
- net +3.3V: now reaches U9.1 (VBAT)
- net +3.3V: now also U9.24 (VDD), U9.36 (VDD), U9.48 (VDD), U9.9 (VDDA), C40.1, C41.1, C42.1, C43.1, C44.1, C45.1, J6.1 (Pin_1), R14.2, R25.2
- net at U9.32 (PA11): now also R23.2
- net at U9.33 (PA12): now also R24.2
- net USB_CONNECT: now reaches U9.38 (PA15)
- new net GND: C40.2, C41.2, C42.2, C43.2, C44.2, C45.2, C46.2, J6.2 (Pin_2)
- new net IF_RESET: C46.1, J6.8 (Pin_8), R14.1
- new net IF_RXD: J6.6 (Pin_6)
- new net IF_SWCLK: J6.3 (Pin_3)
- new net IF_SWO: J6.7 (Pin_7)
- new net IF_TXD: J6.5 (Pin_5)
- new net IF__SWDIO: J6.4 (Pin_4)
- new net TARGET_RESET: R25.1
- new net USB_D+: R24.1
- new net USB_D-: R23.1

Commit message: temp
Parts:
- added C47, C48: 22pF, Capacitor_SMD:C_0603_1608Metric, symbol Device:C
- added J8, J9: Conn_01x03_Pin, Connector_PinHeader_2.54mm:PinHeader_1x03_P2.54mm_Vertical, symbol Connector:Conn_01x03_Pin
- added R26, R27, R28, R29, R30: 22R, Resistor_SMD:R_0805_2012Metric, symbol Device:R
- added R31: 100R, Resistor_SMD:R_0805_2012Metric, symbol Device:R
- added R32, R33: 10k, Resistor_SMD:R_0805_2012Metric, symbol Device:R
- added R34, R35: 10K, Resistor_SMD:R_0805_2012Metric, symbol Device:R
- added Y2: Crystal_GND24, Crystal:Crystal_SMD_3225-4Pin_3.2x2.5mm_HandSoldering, symbol Device:Crystal_GND24
- J6: footprint (none) -> Connector_PinHeader_2.54mm:PinHeader_1x08_P2.54mm_Vertical
- R23, R24: value 100R -> 22R
- SW2: value SW_Push -> SKQGAFE010; footprint Button_Switch_SMD:SW_SPST_B3S-1000 -> Button_Switch_SMD:SW_SPST_SKQG_WithStem
Connections:
- net IF__SWDIO is gone; now on net IF_SWDIO: J6.4 (Pin_4)
- net +3.3V: now also J8.1 (Pin_1), J9.1 (Pin_1)
- net GND: now also SW2.1, U9.23 (VSS), U9.35 (VSS), U9.47 (VSS), U9.8 (VSSA), C47.1, C48.2, J8.3 (Pin_3), J9.3 (Pin_3), Y2.2, Y2.4
- net IF_RESET: now also U9.7 (NRST)
- net IF_RXD: now also U9.31 (PA10)
- net IF_SWCLK: now also U9.37 (PA14)
- net IF_SWO: now also U9.39 (PB3)
- net IF_TXD: now also U9.30 (PA9)
- net TARGET_RESET: now also SW2.2, R26.2
- net TARGET_RXD: now also R28.1
- net TARGET_SWCLK: now also R29.2
- net TARGET_SWDIO: now also R30.2
- net TARGET_TXD: now also R27.1
- net at U9.12 (PA2): now also R27.2
- net at U9.13 (PA3): now also R28.2
- net at U9.18 (PB0): now also R26.1
- net at U9.20 (PB2): now also R33.1
- net at U9.26 (PB13): now also R31.1
- net at U9.27 (PB14): now also R29.1
- net at U9.28 (PB15): now also R30.1, R31.2
- net IF_SWDIO: now reaches U9.34 (PA13)
- net at U9.44 (BOOT0): now also R32.1
- net OSC_IN: now reaches U9.5 (PD0)
- net OSC_IN: now also C47.2, Y2.3
- net OSC_OUT: now reaches U9.6 (PD1)
- net OSC_OUT: now also C48.1, Y2.1
- new net BOOT0: J9.2 (Pin_2), R32.2
- new net BOOT1: J8.2 (Pin_2), R33.2
Other:
- moved on the sheet: C46, J6, R14, R23, R24, SW2

Commit message: temp
Parts:
- removed R34, R35: 10K, Resistor_SMD:R_0805_2012Metric, symbol Device:R
- added C49: 0.1uF, Capacitor_SMD:C_0805_2012Metric, symbol Device:C
- added D10: RUNNING, LED_SMD:LED_0805_2012Metric, symbol Device:LED
- added D11: HID, LED_SMD:LED_0805_2012Metric, symbol Device:LED
- added D12: CDC, LED_SMD:LED_0805_2012Metric, symbol Device:LED
- added D13: MSC, LED_SMD:LED_0805_2012Metric, symbol Device:LED
- added D14: CONNECTED, LED_SMD:LED_0805_2012Metric, symbol Device:LED
- added D8: TX, LED_SMD:LED_0805_2012Metric, symbol Device:LED
- added D9: RX, LED_SMD:LED_0805_2012Metric, symbol Device:LED
- added Q10, Q11: SI2306, Package_TO_SOT_SMD:SOT-23, symbol Transistor_FET:ZXMN3A14F
- added R43, R44: 4.7K, Resistor_SMD:R_0805_2012Metric, symbol Device:R
- added R45: 100R, Resistor_SMD:R_0805_2012Metric, symbol Device:R
- added R46, R47: 100, Resistor_SMD:R_0805_2012Metric, symbol Device:R
- added R48, R49, R50, R51: 470R, Resistor_SMD:R_0805_2012Metric, symbol Device:R
Connections:
- net +3.3V: now also R43.2, R48.1, R49.1
- net GND: now also C49.2, D10.1 (K), D14.1 (K), Q10.2 (S), Q11.2 (S), R44.1
- net IF_RXD: now also R47.1
- net IF_TXD: now also R46.1
- net TARGET_RESET: now also C49.1
- net at U9.26 (PB13): now also R29.1; no longer R31.1
- net at R30.1, R31.2: now also U9.27 (PB14); no longer U9.28 (PB15)
- net at U9.10 (PA0): now also R43.1, R44.2
- net at U9.25 (PB12): now also R31.1
- new net: Q10.1 (G), R46.2
- new net: D8.1 (K), Q10.3 (D)
- new net: Q11.1 (G), R47.2
- new net: D8.2 (A), R49.2
- new net: D10.2 (A), R50.1
- new net: R45.1, U9.28 (PB15)
- new net: D14.2 (A), R51.1
- new net: D9.2 (A), R48.2
- new net: D9.1 (K), Q11.3 (D)
- new net TARGET_SWO: R45.2
Other:
- moved on the sheet: C40, C41, C42, C46, J6, R14, R23, R24, R25, R26, R27, R28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

Commit message: temp
Parts:
- added R52, R53, R54: 1.5k, Resistor_SMD:R_0805_2012Metric, symbol Device:R
Connections:
- net +3.3V: now also D11.2 (A), D12.2 (A), D13.2 (A)
- net at D13.1 (K): now also R54.2
- net LED_nHID: now reaches U9.15 (PA5)
- net LED_nHID: now also R52.1
- net LED_nCDC: now reaches U9.16 (PA6)
- net LED_nCDC: now also R53.1
- net LED_nMSC: now reaches U9.17 (PA7)
- net LED_nMSC: now also R54.1
- net LED_RUNNING: now reaches U9.29 (PA8)
- net LED_RUNNING: now also R50.2
- net LED_CONNECTED: now reaches U9.42 (PB6)
- net LED_CONNECTED: now also R51.2
- net at D11.1 (K): now also R52.2
- net at D12.1 (K): now also R53.2
Other:
- moved on the sheet: D10, D11, D12, D13, D14, R50, R51

Commit message: temp
Parts:
- renumbered C49 to C1, C46 to C10, C47 to C2, C48 to C3, C43 to C4, C44 to C5, C45 to C6, C40 to C7, C41 to C8, C42 to C9, D11 to D1, D12 to D2, D13 to D3, D14 to D4, D10 to D5, D8 to D6, D9 to D7, J8 to J1, J9 to J2, J6 to J3, Q10 to Q1, Q11 to Q2, R52 to R1, R29 to R10, R30 to R11, R31 to R12, R45 to R13, R27 to R14, R28 to R15, R23 to R16, R24 to R17, R43 to R18, R44 to R19, R53 to R2, R46 to R20, R14 to R21, R49 to R22, R47 to R23, R48 to R24, R54 to R3, R25 to R4, R51 to R5, R50 to R6, R32 to R7, R26 to R8, R33 to R9, SW2 to SW1, U9 to U1, Y2 to Y1

Commit message: temp
Parts:
- Y1: footprint Crystal:Crystal_SMD_3225-4Pin_3.2x2.5mm_HandSoldering -> Crystal:Crystal_SMD_3225-4Pin_3.2x2.5mm
Changed lines of the file:
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@@
 			)
 		)
-		(property "Footprint" "Crystal:Crystal_SMD_3225-4Pin_3.2x2.5mm_HandSoldering"
+		(property "Footprint" "Crystal:Crystal_SMD_3225-4Pin_3.2x2.5mm"
 			(at 31.75 78.74 0)
 			(effects

Commit message: temp
Parts:
- removed C4: 0.1uF, Capacitor_SMD:C_0805_2012Metric, symbol Device:C
Changed lines of the file:
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@@
 	)
 	(junction
-		(at 101.6 25.4)
-		(diameter 0)
-		(color 0 0 0 0)
-	)
-	(junction
 		(at 152.4 33.02)
 		(diameter 0)
@@
 	(wire
 		(pts
-			(xy 88.9 25.4) (xy 101.6 25.4)
-		)
-		(stroke
-			(width 0)
-			(type default)
-		)
-	)
-	(wire
-		(pts
 			(xy 133.35 22.86) (xy 133.35 25.4)
 		)
@@
 	(wire
 		(pts
-			(xy 88.9 33.02) (xy 101.6 33.02)
-		)
-		(stroke
-			(width 0)
-			(type default)
-		)
-	)
-	(wire
-		(pts
 			(xy 55.88 149.86) (xy 55.88 151.13)
 		)
@@
 					(unit 1)
 				)
-			)
-		)
-	)
-	(symbol
-		(lib_id "Device:C")
-		(at 88.9 29.21 0)
-		(unit 1)
-		(exclude_from_sim no)
-		(in_bom yes)
-		(on_board yes)
-		(dnp no)
-		(fields_autoplaced yes)
-		(property "Reference" "C4"
-			(at 92.71 27.9399 0)
-			(effects
-				(font
-					(size 1.27 1.27)
-				)
-				(justify left)
-			)
-		)
-		(property "Value" "0.1uF"
-			(at 92.71 30.4799 0)
-			(effects
-				(font
-					(size 1.27 1.27)
-				)
-				(justify left)
-			)
-		)
-		(property "Footprint" "Capacitor_SMD:C_0805_2012Metric"
-			(at 89.8652 33.02 0)
-			(effects
-				(font
-					(size 1.27 1.27)
-				)
-				(hide yes)
-			)
-		)
-		(property "Datasheet" "~"
-			(at 88.9 29.21 0)
-			(effects
-				(font
-					(size 1.27 1.27)
-				)
-				(hide yes)
-			)
-		)
-		(property "Description" "Unpolarized capacitor"
-			(at 88.9 29.21 0)
-			(effects
-				(font
-					(size 1.27 1.27)
-				)
-				(hide yes)
-			)
-		)
-		(pin "2"
-		)
-		(pin "1"
-		)
-		(instances
-			(project "DapLink_STM32F103CBT6"
-				(path "/62d13f52-5b95-4b2e-9bc7-6f5f907932ec/c5505282-deed-4b2e-81f9-216594ebbe5e"
-					(reference "C4")
-					(unit 1)
-				)
