File: Usb.kicad_sch (KiCad schematic)
At the start: 14 parts, among them J4 USB_C_Receptacle_USB2.0_16P, J5 USB4110-GF-A_REVB, Q4 MMBT5401, Q5 MMBT5551L, Q6 DMG2301L, U4 LPC55S69JBD64

Commit message: TEMP
Parts:
- removed Q4: MMBT5401, Package_TO_SOT_SMD:SOT-23, symbol Transistor_BJT:MMBTA92
- removed Q5: MMBT5551L, Package_TO_SOT_SMD:SOT-23, symbol Transistor_BJT:MMBT5551L
- added C28: 0.1uF, Capacitor_SMD:C_0805_2012Metric, symbol Device:C
- added FB1: CBW160808U601T, Inductor_SMD:L_0603_1608Metric, symbol Device:FerriteBead
- added Q4: ZXMN3A14F, Package_TO_SOT_SMD:SOT-23, symbol Transistor_FET:ZXMN3A14F
- added R1: 4.7k, Resistor_SMD:R_0805_2012Metric, symbol Device:R
- added R16, R4: 1.5K, Resistor_SMD:R_0805_2012Metric, symbol Device:R
- added R2, R3: 100R, Resistor_SMD:R_0805_2012Metric, symbol Device:R
- added R21, R22: 5.1k, Resistor_SMD:R_0805_2012Metric, symbol Device:R
- R15: footprint Resistor_SMD:R_0805_2012Metric_Pad1.20x1.40mm_HandSolder -> Resistor_SMD:R_0805_2012Metric
Connections:
- net +3.3V: now also Q6.3 (D), R1.2
- net GND: now also D7.1 (GND), J4.A1 (GND), J4.A12 (GND), J4.B1 (GND), J4.B12 (GND), J4.S1 (SHIELD), C28.2, R21.1, R22.1
- net USB_D+: now also D7.2 (I/O1), J4.A6 (D+), J4.B6 (D+), R15.1, R16.1, R4.1
- net USB_D-: now also D7.3 (I/O2), J4.A7 (D-), J4.B7 (D-)
- net USB_VBUS: now also D7.4 (VCC), J4.A4 (VBUS), J4.A9 (VBUS), J4.B4 (VBUS), J4.B9 (VBUS), C28.1, FB1.1
- net at Q6.1 (G): now also R2.1
- net at Q6.2 (S): now also R4.2
- net at J4.A5 (CC1): now also R22.2
- net at J4.B5 (CC2): now also R21.2
- new net: Q4.1 (G), R3.1
- new net: Q4.3 (D), R1.1, R2.2
- new net +5V: FB1.2
- new net USB_CONNECT: R16.2, R3.2
Other:
- moved on the sheet: D7, Q6, R15
