File: UsbAndPower.kicad_sch (KiCad schematic)
At the start: 28 parts, among them J4 USB_C_Receptacle_USB2.0_16P, Q4 SI2306, Q5 SI2301, U4 LM1117MP-3.3, U5 HT75xx-1-SOT89, U6 RT9193-18GB, U7 RT9193-33GB

Commit message: temp
Parts:
- renumbered C28 to C11, C30 to C12, C32 to C13, C35 to C14, C31 to C15, C34 to C16, C36 to C17, C33 to C18, C37 to C19, C27 to C20, C29 to C21, D7 to D8, Q4 to Q3, Q5 to Q4, R21 to R25, R22 to R26, R16 to R27, R15 to R28, R3 to R29, R1 to R30, R2 to R31, R4 to R32, U4 to U2, U6 to U3, U7 to U4

Commit message: temp
Parts:
- added J7: Conn_01x03_Pin, Connector_PinHeader_2.54mm:PinHeader_1x03_P2.54mm_Vertical, symbol Connector:Conn_01x03_Pin
- added R41, R42: 0R, Resistor_SMD:R_0805_2012Metric, symbol Device:R
Connections:
- net +3.3V_LDO is gone; now on net +3.3V: C19.1, U4.5 (OUT)
- net +1.8V_LDO: now also J7.3 (Pin_3), R41.2
- new net +1.8V: J7.2 (Pin_2), R41.1, R42.2
- new net +1.8V_Target: J7.1 (Pin_1), R42.1
