File: DapLink_STM32F103CBT6.kicad_pcb (KiCad board)
At the start: 2 copper layers, 154 x 97.5 mm, 105 parts, among them J4 USB_C_Receptacle_USB2.0_16P, J5 Conn_01x08_Pin, J6 Conn_01x08_Pin, J7 Conn_01x08_Pin, J8 Conn_01x03_Pin, J9 Conn_01x03_Pin, Q4 ZXMN3A14F, Q6 DMG2301L, SW2 SKQGAFE010, U4 LM1117MP-3.3, U5 HT75xx-1-SOT89, U6 RT9193-18GB, U7 RT9193-33GB, U8 TXB0104PW, U9 STM32F103CBTx

Commit message: temp
Parts:
- removed C24: 8p, Capacitor_SMD:C_0402_1005Metric
- removed C25: 100n, Capacitor_SMD:C_0402_1005Metric
- removed C26: 22u, Capacitor_SMD:C_0402_1005Metric
- removed C27, C30: 10uF 10V, Capacitor_SMD:C_0805_2012Metric
- removed C28, C38, C39, C40, C41, C42, C43, C44, C46: 0.1uF, Capacitor_SMD:C_0805_2012Metric
- removed C29, C31: 10uF 6.3V, Capacitor_SMD:C_0805_2012Metric
- removed C32, C33, C35, C37, C45: 1uF 10V X7R, Capacitor_SMD:C_1206_3216Metric
- removed C34, C36: 22nF, Capacitor_SMD:C_0805_2012Metric
- removed J8, J9: Conn_01x03_Pin, Connector_PinHeader_2.54mm:PinHeader_1x03_P2.54mm_Vertical
- removed JP1: SWD disable, Jumper:SolderJumper-2_P1.3mm_Open_RoundedPad1.0x1.5mm
- removed L2, L3, L4: MI0603J601R-10, Inductor_SMD:L_0603_1608Metric
- removed L5: 4u7, Inductor_SMD:L_0603_1608Metric
- removed SW2: SKQGAFE010, Button_Switch_SMD:SW_SPST_SKQG_WithStem
- removed U7: RT9193-33GB, Package_TO_SOT_SMD:SOT-23-5
- removed U8: TXB0104PW, Package_SO:TSSOP-14_4.4x5mm_P0.65mm
- removed U9: STM32F103CBTx, Package_QFP:LQFP-48_7x7mm_P0.5mm
- added D1: HID, LED_SMD:LED_0805_2012Metric, F.Cu at (37.0, 25.0)
- added D6: TX, LED_SMD:LED_0805_2012Metric, F.Cu at (37.0, 25.0)
- added D8: PRTR5V0U2X, Package_TO_SOT_SMD:SOT-143, F.Cu at (187.0, 102.0)
- added H1: M3-3.2mm, MountingHole:MountingHole_3.2mm_M3_Pad_Via, F.Cu at (168.1, 32.6)
- added H2: M3-3.2mm, MountingHole:MountingHole_3.2mm_M3_Pad_Via, F.Cu at (168.1, 40.6)
- added H3: M3-3.2mm, MountingHole:MountingHole_3.2mm_M3_Pad_Via, F.Cu at (168.1, 48.5)
- added H4: M3-3.2mm, MountingHole:MountingHole_3.2mm_M3_Pad_Via, F.Cu at (168.1, 56.5)
- added J1: Conn_01x03_Pin, Connector_PinHeader_2.54mm:PinHeader_1x03_P2.54mm_Vertical, F.Cu at (45.0, 105.0)
- added J2: Conn_01x03_Pin, Connector_PinHeader_2.54mm:PinHeader_1x03_P2.54mm_Vertical, F.Cu at (121.0, 39.0)
- added J3: Conn_01x08_Pin, Connector_PinHeader_2.54mm:PinHeader_1x08_P2.54mm_Vertical, F.Cu at (153.0, 90.0)
- added Q1: SI2306, Package_TO_SOT_SMD:SOT-23, F.Cu at (142.0, 28.0)
- added Q2: SI2306, Package_TO_SOT_SMD:SOT-23, F.Cu at (190.0, 65.0)
- added Q3: SI2306, Package_TO_SOT_SMD:SOT-23, F.Cu at (187.0, 96.0)
- added Q5: SI2306, Package_TO_SOT_SMD:SOT-23, F.Cu at (70.0, 84.0)
- added Q7: SI2306, Package_TO_SOT_SMD:SOT-23, F.Cu at (108.0, 116.0)
- added Q8: SI2306, Package_TO_SOT_SMD:SOT-23, F.Cu at (142.0, 114.0)
- added R34: 100K, Resistor_SMD:R_0805_2012Metric, F.Cu at (118.0, 91.0)
- added R35, R36: 100K, Resistor_SMD:R_0805_2012Metric, F.Cu at (37.0, 25.0)
- added R37: 4.7K, Resistor_SMD:R_0805_2012Metric, F.Cu at (190.0, 85.0)
- added R38, R43: 100R, Resistor_SMD:R_0805_2012Metric, F.Cu at (37.0, 25.0)
- added R39: 10K, Resistor_SMD:R_0805_2012Metric, F.Cu at (110.0, 28.0)
- added R40: 10K, Resistor_SMD:R_0805_2012Metric, F.Cu at (140.0, 34.0)
- added R41: 0R, Resistor_SMD:R_0805_2012Metric, F.Cu at (125.0, 121.0)
- added R42: 0R, Resistor_SMD:R_0805_2012Metric, F.Cu at (171.0, 119.0)
- added R44: 10K, Resistor_SMD:R_0805_2012Metric, F.Cu at (144.0, 119.0)
- added R45: 4.7K, Resistor_SMD:R_0805_2012Metric, F.Cu at (37.0, 25.0)
- added SW1: SKQGAFE010, Button_Switch_SMD:SW_SPST_SKQG_WithStem, F.Cu at (46.0, 85.0)
- added U1: STM32F103CBTx, Package_QFP:LQFP-48_7x7mm_P0.5mm, F.Cu at (45.0, 56.0)
- added U2: LM1117MP-3.3, Package_TO_SOT_SMD:SOT-223-3_TabPin2, F.Cu at (86.0, 107.0)
- added U3: RT9193-18GB, Package_TO_SOT_SMD:SOT-23-5, F.Cu at (189.0, 90.0)
- added Y1: Crystal_GND24, Crystal:Crystal_SMD_3225-4Pin_3.2x2.5mm_HandSoldering, F.Cu at (66.0, 33.0)
- C1, C10: value 10u -> 0.1uF; footprint Capacitor_SMD:C_0402_1005Metric -> Capacitor_SMD:C_0805_2012Metric
- C11, C4, C5, C7, C8, C9: value 100n -> 0.1uF; footprint Capacitor_SMD:C_0402_1005Metric -> Capacitor_SMD:C_0805_2012Metric
- C12: value 10n -> 10uF 10V; footprint Capacitor_SMD:C_0402_1005Metric -> Capacitor_SMD:C_0805_2012Metric
- C13, C14, C6: value 10n -> 1uF 10V X7R; footprint Capacitor_SMD:C_0402_1005Metric -> Capacitor_SMD:C_1206_3216Metric
- C15: value 22u -> 10uF 6.3V; footprint Capacitor_SMD:C_0402_1005Metric -> Capacitor_SMD:C_0805_2012Metric
- C16: value 10n -> 22nF; footprint Capacitor_SMD:C_0402_1005Metric -> Capacitor_SMD:C_0805_2012Metric
- C17: value 100n -> 22nF; footprint Capacitor_SMD:C_0402_1005Metric -> Capacitor_SMD:C_0805_2012Metric
- C18: value 100n -> 1uF 10V X7R; footprint Capacitor_SMD:C_0402_1005Metric -> Capacitor_SMD:C_1206_3216Metric
- C19: value 47p -> 1uF 10V X7R; footprint Capacitor_SMD:C_0402_1005Metric -> Capacitor_SMD:C_1206_3216Metric
- C2: value 100n -> 22pF; footprint Capacitor_SMD:C_0402_1005Metric -> Capacitor_SMD:C_0603_1608Metric
- C20: value 47p -> 10uF 10V; footprint Capacitor_SMD:C_0402_1005Metric -> Capacitor_SMD:C_0805_2012Metric
- C21: value 8p -> 10uF 6.3V; footprint Capacitor_SMD:C_0402_1005Metric -> Capacitor_SMD:C_0805_2012Metric
- C22: value 22u -> 0.1uF; footprint Capacitor_SMD:C_0402_1005Metric -> Capacitor_SMD:C_0805_2012Metric
- C23: value 47p -> 0.1uF; footprint Capacitor_SMD:C_0402_1005Metric -> Capacitor_SMD:C_0805_2012Metric
- C3: value 4u7 -> 22pF; footprint Capacitor_SMD:C_0402_1005Metric -> Capacitor_SMD:C_0603_1608Metric
- D2: value PESD5V0L5UV -> CDC; footprint Package_TO_SOT_SMD:SOT-666 -> LED_SMD:LED_0805_2012Metric
- D3: value LED_RED -> MSC; footprint LED_SMD:LED_0402_1005Metric -> LED_SMD:LED_0805_2012Metric
- D4: value PMEG3005AESFYL -> CONNECTED; footprint Diode_SMD:Nexperia_DSN0603-2_0.6x0.3mm_P0.4mm -> LED_SMD:LED_0805_2012Metric
- D5: value PESD5V0L5UV -> RUNNING; footprint Package_TO_SOT_SMD:SOT-666 -> LED_SMD:LED_0805_2012Metric
- D7: value PRTR5V0U2X -> RX; footprint Package_TO_SOT_SMD:SOT-143 -> LED_SMD:LED_0805_2012Metric
- J7: value Conn_01x08_Pin -> Conn_01x03_Pin; footprint Connector_PinHeader_2.54mm:PinHeader_1x08_P2.54mm_Vertical -> Connector_PinHeader_2.54mm:PinHeader_1x03_P2.54mm_Vertical
- Q4: value ZXMN3A14F -> SI2301
- Q6: value DMG2301L -> SI2306
- R1: value 4.7k -> 1.5k
- R10: value 2k -> 22R; footprint Resistor_SMD:R_0402_1005Metric -> Resistor_SMD:R_0805_2012Metric
- R11: value 100 -> 22R; footprint Resistor_SMD:R_0402_1005Metric -> Resistor_SMD:R_0805_2012Metric
- R12: value 100K -> 100R
- R13: value 10K -> 100R
- R14: value 10K -> 22R
- R15, R16: value 1.5K -> 22R
- R17: value 100k -> 22R; footprint Resistor_SMD:R_0402_1005Metric -> Resistor_SMD:R_0805_2012Metric
- R18: value 100k -> 4.7K; footprint Resistor_SMD:R_0402_1005Metric -> Resistor_SMD:R_0805_2012Metric
- R19: value 2k -> 4.7K; footprint Resistor_SMD:R_0402_1005Metric -> Resistor_SMD:R_0805_2012Metric
- R2, R3: value 100R -> 1.5k
- R20: value 10 -> 100; footprint Resistor_SMD:R_0402_1005Metric -> Resistor_SMD:R_0805_2012Metric
- R21: value 5.1k -> 10K
- R22: value 5.1k -> 470R
- R23: value 22R -> 100
- R24: value 22R -> 470R
- R25: value 10K -> 5.1k
- R26: value 22R -> 5.1k
- R27, R28: value 22R -> 1.5K
- R29: value 22R -> 100R
- R30: value 22R -> 4.7k
- R32: value 10k -> 1.5K
- R33: value 10k -> 10K
- R4: value 1.5K -> 10K
- R5, R6: value 5k1 -> 470R; footprint Resistor_SMD:R_0402_1005Metric -> Resistor_SMD:R_0805_2012Metric
- R7, R9: footprint Resistor_SMD:R_0402_1005Metric -> Resistor_SMD:R_0805_2012Metric
- R8: value 20k -> 22R; footprint Resistor_SMD:R_0402_1005Metric -> Resistor_SMD:R_0805_2012Metric
- U4: value LM1117MP-3.3 -> RT9193-33GB; footprint Package_TO_SOT_SMD:SOT-223-3_TabPin2 -> Package_TO_SOT_SMD:SOT-23-5
- U6: value RT9193-18GB -> TXB0104PW; footprint Package_TO_SOT_SMD:SOT-23-5 -> Package_SO:TSSOP-14_4.4x5mm_P0.65mm
- moved R26 86.0 mm to (64.5, 117.0), turned to -90 degrees
- moved R25 71.3 mm to (79.0, 117.0), turned to -90 degrees
- moved J4 33.5 mm to (72.0, 119.5)
Connections:
- C1 pad 1: +5V -> /Mcu/TARGET_RESET
- C10 pad 1: +3V3 -> /Mcu/IF_RESET
- C11 pad 1: /MCU-LINK Power and USB/MCU_VDDIO -> /UsbAndPower/USB_VBUS
- C12 pad 1: /MCU-LINK Power and USB/MCU_VDDIO -> +5V
- C13 pad 1: /MCU-LINK Power and USB/MCU_VDDIO -> +5V
- C14 pad 1: /MCU-LINK Power and USB/MCU_VDDIO -> +5V
- C15 pad 1: Net-(U2A-VBAT_DCDC) -> +3.3V
- C16 pad 1: /MCU-LINK Power and USB/MCU_VDDIO -> Net-(U3-BP)
- C17 pad 1: +3V3 -> Net-(U4-BP)
- C18 pad 1: Net-(U2A-VBAT_DCDC) -> +1.8V_LDO
- C19 pad 1: +3V3 -> +3.3V_LDO
- C2 pad 1: +5V -> GND
- C2 pad 2: GND -> /Mcu/OSC_IN
- C20 pad 1: Net-(U2A-VBAT_DCDC) -> +5V
- C21 pad 1: /MCU-LINK Power and USB/Q- -> +3.3V
- C22 pad 1: Net-(U2A-FB) -> +1.8V
- C23 pad 1: Net-(U2A-FB) -> +3.3V
- C3 pad 1: /MCU-LINK Power and USB/MCU_VDDIO -> /Mcu/OSC_OUT
- C4 pad 1: /MCU-LINK Power and USB/MCU_VDDIO -> +3.3V
- C5 pad 1: /MCU-LINK Power and USB/MCU_VDDIO -> +3.3V
- C6 pad 1: /MCU-LINK Power and USB/USB_VBUS -> +3.3V
- C7 pad 1: /MCU-LINK Power and USB/MCU_VDDIO -> +3.3V
- C8 pad 1: +3V3 -> +3.3V
- C9 pad 1: /MCU-LINK Power and USB/MCU_VDDIO -> +3.3V
- D2 pad 1: /Debug and UART Interface/TARGET_SWDIO -> Net-(D2-K)
- D2 pad 2: GND -> +3.3V
- D3 pad 1: /Debug and UART Interface/PIO0_5-ISP_EN-LED1_CTRL -> Net-(D3-K)
- D3 pad 2: Net-(D3-A) -> +3.3V
- D4 pad 1: /Debug and UART Interface/VCC -> GND
- D5 pad 1: Net-(D5A-K1) -> GND
- D5 pad 2: GND -> Net-(D5-A)
- D7 pad 1: GND -> Net-(D7-K)
- D7 pad 2: /UsbAndPower/USB_D+ -> Net-(D7-A)
- J5 pad 1: +1.8V -> +3.3V
- J5 pad 3: /DebugAndUart/TARGET_1v8_SWCLK -> /DebugAndUart/TARGET_SWCLK
- J5 pad 4: /DebugAndUart/TARGET_1v8_SWDIO -> /DebugAndUart/TARGET_SWDIO
- J5 pad 5: /DebugAndUart/TARGET_1v8_TXD -> /DebugAndUart/TARGET_TXD
- J5 pad 6: /DebugAndUart/TARGET_1v8_RXD -> /DebugAndUart/TARGET_RXD
- J5 pad 7: /DebugAndUart/TARGET_1v8_SWO -> /DebugAndUart/TARGET_SWO
- J5 pad 8: /DebugAndUart/TARGET_1v8_RESET -> /DebugAndUart/TARGET_RESET
- J6 pad 1: +3.3V -> +1.8V_Target
- J6 pad 3: /Mcu/IF_SWCLK -> /DebugAndUart/TARGET_1v8_SWCLK
- J6 pad 4: /Mcu/IF_SWDIO -> /DebugAndUart/TARGET_1v8_SWDIO
- J6 pad 5: /Mcu/IF_TXD -> /DebugAndUart/TARGET_1v8_TXD
- J6 pad 6: /Mcu/IF_RXD -> /DebugAndUart/TARGET_1v8_RXD
- J6 pad 7: /Mcu/IF_SWO -> /DebugAndUart/TARGET_1v8_SWO
- J6 pad 8: /Mcu/IF_RESET -> /DebugAndUart/TARGET_1v8_RESET
- J7 pad 1: +3.3V -> +1.8V_Target
- J7 pad 2: GND -> +1.8V
- J7 pad 3: /DebugAndUart/TARGET_SWCLK -> +1.8V_LDO
- Q4 pad 2: GND -> +3.3V
- Q6 pad 1: Net-(Q6-G) -> Net-(Q5-D)
- Q6 pad 2: Net-(Q6-S) -> GND
- Q6 pad 3: +3.3V -> /DebugAndUart/TARGET_SWO
- R1 pad 1: Net-(Q4-D) -> /Mcu/LED_nHID
- R1 pad 2: +3.3V -> Net-(D1-K)
- R10 pad 1: +3V3 -> Net-(U1-PB13)
- R10 pad 2: Net-(D3-A) -> /Mcu/TARGET_SWCLK
- R11 pad 1: Net-(D2C-K3) -> Net-(U1-PB14)
- R11 pad 2: /Debug and UART Interface/TARGET_SWO -> /Mcu/TARGET_SWDIO
- R12 pad 1: GND -> Net-(U1-PB12)
- R12 pad 2: Net-(U8-OE) -> Net-(U1-PB14)
- R13 pad 1: Net-(U8-OE) -> Net-(U1-PB15)
- R13 pad 2: +1.8V -> /Mcu/TARGET_SWO
- R14 pad 1: /Mcu/IF_RESET -> /Mcu/TARGET_TXD
- R14 pad 2: +3.3V -> Net-(U1-PA2)
- R15 pad 1: /UsbAndPower/USB_D+ -> /Mcu/TARGET_RXD
- R15 pad 2: +3.3V -> Net-(U1-PA3)
- R16 pad 1: /UsbAndPower/USB_D+ -> /Mcu/USB_D-
- R16 pad 2: /UsbAndPower/USB_CONNECT -> Net-(U1-PA11)
- R17 pad 1: /Debug and UART Interface/TARGET_SWCLK -> /Mcu/USB_D+
- R17 pad 2: GND -> Net-(U1-PA12)
- R18 pad 1: +3V3 -> Net-(U1-PA0)
- R18 pad 2: /Debug and UART Interface/TARGET_SWDIO -> +3.3V
- R19 pad 1: /Debug and UART Interface/TARGET_DETECT -> GND
- R19 pad 2: Net-(D5A-K1) -> Net-(U1-PA0)
- R2 pad 1: Net-(Q6-G) -> /Mcu/LED_nCDC
- R2 pad 2: Net-(Q4-D) -> Net-(D2-K)
- R20 pad 1: /Debug and UART Interface/TARGET_ISP_CTRL -> /Mcu/IF_TXD
- R20 pad 2: Net-(D5B-K2) -> Net-(Q1-G)
- R21 pad 1: GND -> /Mcu/IF_RESET
- R21 pad 2: Net-(J4-CC2) -> +3.3V
- R22 pad 1: GND -> +3.3V
- R22 pad 2: Net-(J4-CC1) -> Net-(D6-A)
- R23 pad 1: /Mcu/USB_D- -> /Mcu/IF_RXD
- R24 pad 1: /Mcu/USB_D+ -> +3.3V
- R24 pad 2: Net-(U9-PA12) -> Net-(D7-A)
- R25 pad 1: /Mcu/TARGET_RESET -> GND
- R25 pad 2: +3.3V -> Net-(J4-CC2)
- R26 pad 1: Net-(U9-PB0) -> GND
- R26 pad 2: /Mcu/TARGET_RESET -> Net-(J4-CC1)
- R27 pad 1: /Mcu/TARGET_TXD -> /UsbAndPower/USB_D+
- R27 pad 2: Net-(U9-PA2) -> /UsbAndPower/USB_CONNECT
- R28 pad 1: /Mcu/TARGET_RXD -> /UsbAndPower/USB_D+
- R28 pad 2: Net-(U9-PA3) -> +3.3V
- R29 pad 2: /Mcu/TARGET_SWCLK -> /UsbAndPower/USB_CONNECT
- R3 pad 1: Net-(Q4-G) -> /Mcu/LED_nMSC
- R3 pad 2: /UsbAndPower/USB_CONNECT -> Net-(D3-K)
- R30 pad 2: /Mcu/TARGET_SWDIO -> +3.3V
- R31 pad 1: Net-(U9-PB13) -> Net-(Q4-G)
- R32 pad 1: Net-(U9-BOOT0) -> /UsbAndPower/USB_D+
- R32 pad 2: /Mcu/BOOT0 -> Net-(Q4-D)
- R33 pad 1: Net-(U9-PB2) -> Net-(U6-OE)
- R33 pad 2: /Mcu/BOOT1 -> +1.8V
- R4 pad 1: /UsbAndPower/USB_D+ -> /Mcu/TARGET_RESET
- R4 pad 2: Net-(Q6-S) -> +3.3V
- R5 pad 1: GND -> Net-(D4-A)
- R5 pad 2: Net-(J1-CC2) -> /Mcu/LED_CONNECTED
- R6 pad 1: GND -> Net-(D5-A)
- R6 pad 2: Net-(J1-CC1) -> /Mcu/LED_RUNNING
- R7 pad 1: Net-(U2B-USB1_VBUS) -> Net-(U1-BOOT0)
- R7 pad 2: +5V -> /Mcu/BOOT0
- R8 pad 1: GND -> Net-(U1-PB0)
- R8 pad 2: Net-(U2B-USB1_VBUS) -> /Mcu/TARGET_RESET
- R9 pad 1: +5V -> Net-(U1-PB2)
- R9 pad 2: GND -> /Mcu/BOOT1
- U4 pad 1: GND -> +5V
- U4 pad 2: +3.3V -> GND
- U6 pad 1: +5V -> +1.8V
- U6 pad 2: GND -> /DebugAndUart/TARGET_1v8_SWCLK
- U6 pad 3: +5V -> /DebugAndUart/TARGET_1v8_SWDIO
- U6 pad 4: Net-(U6-BP) -> /DebugAndUart/TARGET_1v8_TXD
- U6 pad 5: +1.8V -> /DebugAndUart/TARGET_1v8_RXD

Commit message: temp
Parts:
- moved C11 145.4 mm to (48.3, 85.3), turned to -90 degrees
- moved C13 141.0 mm to (51.4, 139.2)
- moved U3 137.1 mm to (60.4, 137.6)
- moved C16 135.1 mm to (59.0, 145.1)
- moved FB1 77.6 mm to (50.5, 85.3), turned to -90 degrees
- moved C10 69.5 mm to (112.9, 43.6)
- moved D2 69.5 mm to (113.9, 59.6)
- moved J1 69.5 mm to (93.9, 55.6)
- moved R21 69.5 mm to (92.9, 72.6)
- moved R3 69.5 mm to (92.9, 68.6)
- moved SW1 69.5 mm to (94.9, 35.6)
- moved R25 56.5 mm to (42.4, 74.0), turned to 0 degrees
- moved C18 55.2 mm to (68.3, 143.0)
- moved J4 48.3 mm to (42.2, 81.5), turned to -90 degrees
- moved R26 46.6 mm to (46.6, 74.0), turned to 180 degrees
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Routing:
- net Net-(J4-CC2): track 0.00 -> 11.7 mm
- net Net-(J4-CC1): track 0.00 -> 9.62 mm
- net /UsbAndPower/USB_VBUS: track 0.00 -> 1.88 mm, vias 0 -> 1

Commit message: temp
Parts:
- moved R31 174.1 mm to (21.6, 39.3)
- moved Q3 170.3 mm to (26.2, 40.0), turned to 180 degrees
- moved R36 168.0 mm to (116.1, 173.2), turned to 90 degrees
- moved R32 167.5 mm to (26.0, 43.1), turned to 180 degrees
- moved R33 165.2 mm to (108.4, 174.0), turned to 180 degrees
- moved R35 162.3 mm to (116.1, 166.7), turned to 90 degrees
- moved C22 157.9 mm to (108.0, 166.0)
- moved C14 145.4 mm to (46.5, 96.3), turned to -90 degrees
- moved U6 100.6 mm to (110.1, 170.1)
- moved R41 95.0 mm to (193.4, 55.1), turned to -90 degrees
- moved C23 93.2 mm to (112.3, 166.0), turned to 180 degrees
- moved C15 85.3 mm to (98.7, 105.8), turned to 90 degrees
- moved R34 83.2 mm to (112.3, 174.0), turned to 180 degrees
- moved C21 77.5 mm to (61.7, 98.5), turned to 90 degrees
- moved R42 72.6 mm to (193.4, 49.9), turned to -90 degrees
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Connections:
- C19 pad 1: +3.3V_LDO -> +3.3V
- U4 pad 5: +3.3V_LDO -> +3.3V
Routing:
- net +3.3V: track 0.00 -> 6.92 mm
- net Net-(Q3-D): track 0.00 -> 5.25 mm
- net +5V: track 0.00 -> 3.15 mm
- net Net-(Q4-D): track 0.00 -> 2.58 mm
- net Net-(Q4-G): track 0.00 -> 2.15 mm

Commit message: temp
Parts:
- Y1: footprint Crystal:Crystal_SMD_3225-4Pin_3.2x2.5mm_HandSoldering -> Crystal:Crystal_SMD_3225-4Pin_3.2x2.5mm
- moved C4 413.4 mm to (502.4, 174.3)
- moved C9 413.4 mm to (600.3, 168.2)
- moved R9 394.8 mm to (427.2, 85.0)
- moved R7 388.9 mm to (422.3, 77.8)
- moved R19 387.9 mm to (420.1, 86.0)
- moved R16 386.0 mm to (469.9, 76.2)
- moved R4 386.0 mm to (429.9, 76.2)
- moved SW1 386.0 mm to (477.8, 83.8)
- moved R17 385.3 mm to (418.5, 78.9)
- moved C1 383.2 mm to (416.9, 75.4)
- moved R8 379.4 mm to (412.7, 77.7)
- moved R18 374.5 mm to (406.9, 83.5)
- moved C10 274.5 mm to (366.7, -60.8)
- moved D2 274.5 mm to (367.7, -44.8)
- moved D4 274.5 mm to (377.8, 5.60)
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Connections:
- C1 pad 1: /Mcu/TARGET_RESET -> /DebugAndUart/TARGET_RESET
- R10 pad 2: /Mcu/TARGET_SWCLK -> /DebugAndUart/TARGET_SWCLK
- R11 pad 2: /Mcu/TARGET_SWDIO -> /DebugAndUart/TARGET_SWDIO
- R13 pad 2: /Mcu/TARGET_SWO -> /DebugAndUart/TARGET_SWO
- R14 pad 1: /Mcu/TARGET_TXD -> /DebugAndUart/TARGET_TXD
- R15 pad 1: /Mcu/TARGET_RXD -> /DebugAndUart/TARGET_RXD
- R16 pad 1: /Mcu/USB_D- -> /UsbAndPower/USB_D-
- R17 pad 1: /Mcu/USB_D+ -> /UsbAndPower/USB_D+
- R4 pad 1: /Mcu/TARGET_RESET -> /DebugAndUart/TARGET_RESET
- R8 pad 2: /Mcu/TARGET_RESET -> /DebugAndUart/TARGET_RESET
- SW1 pad 2: /Mcu/TARGET_RESET -> /DebugAndUart/TARGET_RESET
- U1 pad 38: /Mcu/USB_CONNECT -> /UsbAndPower/USB_CONNECT
- U6 pad 10: /DebugAndUart/TARGET_RXD -> /DebugAndUart/TARGET_SWCLK
- U6 pad 11: /DebugAndUart/TARGET_TXD -> /DebugAndUart/TARGET_SWDIO
- U6 pad 12: /DebugAndUart/TARGET_SWDIO -> /DebugAndUart/TARGET_TXD
- U6 pad 13: /DebugAndUart/TARGET_SWCLK -> /DebugAndUart/TARGET_RXD
- U6 pad 2: /DebugAndUart/TARGET_1v8_SWCLK -> /DebugAndUart/TARGET_1v8_RXD
- U6 pad 3: /DebugAndUart/TARGET_1v8_SWDIO -> /DebugAndUart/TARGET_1v8_TXD
- U6 pad 4: /DebugAndUart/TARGET_1v8_TXD -> /DebugAndUart/TARGET_1v8_SWDIO
- U6 pad 5: /DebugAndUart/TARGET_1v8_RXD -> /DebugAndUart/TARGET_1v8_SWCLK
Routing:
- net Net-(U1-PB14): track 0.00 -> 12.4 mm, vias 0 -> 2
- net Net-(U1-PB15): track 0.00 -> 8.34 mm
- net GND: track 0.00 -> 8.02 mm, vias 0 -> 2
- net Net-(U1-PB13): track 0.00 -> 7.89 mm
- net /Mcu/OSC_IN: track 0.00 -> 7.45 mm
- net /Mcu/OSC_OUT: track 0.00 -> 7.10 mm
- net Net-(U1-PB12): track 0.00 -> 3.41 mm
- net +3.3V: track 6.92 -> 10.2 mm
- net /Mcu/IF_RESET: track 0.00 -> 1.93 mm, vias 0 -> 1

Commit message: temp
Parts:
- moved SW1 404.8 mm to (73.6, 61.8)
- moved R16 396.0 mm to (74.0, 80.4)
- moved R4 352.7 mm to (77.4, 66.0)
- moved C1 349.4 mm to (67.8, 61.5), turned to 90 degrees
- moved C9 345.0 mm to (255.9, 148.6)
- moved R17 344.5 mm to (74.0, 82.5)
- moved R7 342.2 mm to (82.2, 40.0)
- moved R9 336.0 mm to (94.1, 41.3), turned to 90 degrees
- moved R18 334.4 mm to (73.0, 66.2)
- moved R8 315.4 mm to (98.0, 98.2)
- moved D2 310.6 mm to (96.0, 105.6), turned to -90 degrees
- moved J3 309.4 mm to (106.2, 58.8), turned to -90 degrees
- moved J2 306.5 mm to (86.5, 38.6)
- moved R3 283.3 mm to (99.0, 101.7), turned to -90 degrees
- moved J7 278.5 mm to (97.9, 135.5)
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Routing:
- net GND: track 8.02 -> 40.3 mm, vias 2 -> 6
- net +5V: track 3.15 -> 11.2 mm
- net Net-(Q7-D): track 0.00 -> 5.56 mm
- net /DebugAndUart/TARGET_1v8_RESET: track 0.00 -> 3.70 mm
- net Net-(Q7-G): track 0.00 -> 2.96 mm
- net +1.8V_LDO: track 0.00 -> 2.49 mm
- net +3.3V: track 10.2 -> 12.6 mm
- net /UsbAndPower/USB_D+: track 0.00 -> 2.20 mm
- net Net-(U3-BP): track 0.00 -> 2.20 mm
- net /UsbAndPower/USB_CONNECT: track 0.00 -> 2.17 mm
- net Net-(U4-BP): track 0.00 -> 2.13 mm

Commit message: temp
Parts:
- removed C4: 0.1uF, Capacitor_SMD:C_0805_2012Metric
- moved C10 261.2 mm to (81.9, 72.8), turned to 180 degrees
- moved R21 228.6 mm to (85.8, 72.9)
- moved D4 223.3 mm to (113.8, 75.3), turned to 180 degrees
- moved C9 178.5 mm to (90.1, 82.5), turned to 180 degrees
- moved R6 159.7 mm to (110.1, 78.0), turned to 180 degrees
- moved R5 157.9 mm to (110.1, 75.3), turned to 180 degrees
- moved D5 146.0 mm to (113.8, 78.0), turned to 180 degrees
- moved R19 140.9 mm to (86.0, 97.7)
- moved J7 75.7 mm to (138.8, 71.8), turned to -90 degrees
- moved R41 73.0 mm to (133.7, 75.2), turned to 180 degrees
- moved R42 71.0 mm to (138.9, 75.2), turned to 180 degrees
- moved R18 31.7 mm to (87.6, 94.2)
- moved R40 24.1 mm to (130.7, 96.5), turned to 0 degrees
- moved Q6 19.2 mm to (134.6, 99.4), turned to 180 degrees
- moved R39 19.1 mm to (134.8, 96.5), turned to 180 degrees
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Routing:
- net GND: track 40.3 -> 67.4 mm, vias 6 -> 7
- net /DebugAndUart/TARGET_RXD: track 0.00 -> 11.4 mm
- net /DebugAndUart/TARGET_TXD: track 0.00 -> 10.9 mm
- net +1.8V: track 0.00 -> 10.6 mm, vias 0 -> 2
- net /DebugAndUart/TARGET_SWCLK: track 0.00 -> 9.90 mm
- net /DebugAndUart/TARGET_SWDIO: track 0.00 -> 9.16 mm
- net /DebugAndUart/TARGET_1v8_RXD: track 0.00 -> 8.74 mm
- net /DebugAndUart/TARGET_1v8_TXD: track 0.00 -> 7.94 mm
- net /DebugAndUart/TARGET_1v8_SWCLK: track 0.00 -> 7.90 mm
- net /DebugAndUart/TARGET_1v8_SWDIO: track 0.00 -> 7.16 mm
- net Net-(U6-OE): track 0.00 -> 5.74 mm

Commit message: TEMP
Parts:
- moved R8 24.2 mm to (118.0, 111.8)
- moved C2 12.3 mm to (95.7, 88.0)
- moved C3 12.3 mm to (96.3, 92.2)
- moved C5 12.3 mm to (112.8, 96.2)
- moved C6 12.3 mm to (102.6, 83.5)
- moved C7 12.3 mm to (101.0, 92.0)
- moved C8 12.3 mm to (114.3, 83.8)
- moved C9 12.3 mm to (102.0, 85.8)
- moved D1 12.3 mm to (104.9, 108.8)
- moved D2 12.3 mm to (107.9, 108.8)
- moved D3 12.3 mm to (110.9, 108.8)
- moved R1 12.3 mm to (104.9, 105.0)
- moved R12 12.3 mm to (117.0, 93.5)
- moved R18 12.3 mm to (99.5, 97.5)
- moved R19 12.3 mm to (97.9, 101.0)
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Routing:
- net /DebugAndUart/TARGET_SWO: track 0.00 -> 22.0 mm, vias 0 -> 1
- net Net-(Q5-D): track 0.00 -> 6.52 mm
- net /DebugAndUart/TARGET_1v8_SWO: track 0.00 -> 6.10 mm
- net Net-(Q5-G): track 0.00 -> 4.60 mm
- net /DebugAndUart/TARGET_SWCLK: track 9.90 -> 14.0 mm
- net /DebugAndUart/TARGET_1v8_RESET: track 3.70 -> 0.00 mm
- net GND: track 67.4 -> 63.8 mm
- net /DebugAndUart/TARGET_SWDIO: track 9.16 -> 12.7 mm
- net Net-(Q7-D): track 5.56 -> 8.14 mm
- net Net-(U1-PB14): track 12.3 -> 10.1 mm
- net /DebugAndUart/TARGET_RXD: track 11.4 -> 9.55 mm
- net /DebugAndUart/TARGET_TXD: track 10.9 -> 9.19 mm
- net /DebugAndUart/TARGET_1v8_TXD: track 7.94 -> 6.40 mm
- net /DebugAndUart/TARGET_1v8_SWDIO: track 7.16 -> 5.66 mm
- net /DebugAndUart/TARGET_1v8_SWCLK: track 7.90 -> 6.44 mm
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
Commit message: reasonable placement for pcb
Parts:
- moved C12 83.0 mm to (30.6, 32.1)
- moved C15 83.0 mm to (40.5, 36.9)
- moved U2 83.0 mm to (35.5, 34.3)
- moved C20 61.1 mm to (42.2, 42.6)
- moved C21 61.1 mm to (34.2, 43.9)
- moved U5 61.1 mm to (38.5, 43.4)
- moved R21 48.7 mm to (55.5, 50.2), turned to 90 degrees
- moved R19 48.3 mm to (51.7, 115.1)
- moved R18 47.5 mm to (55.4, 115.1)
- moved Q1 44.2 mm to (72.6, 60.1)
- moved D6 44.2 mm to (72.6, 56.4)
- moved R22 44.2 mm to (70.6, 56.4)
- moved R20 44.2 mm to (69.9, 60.3)
- moved J7 44.1 mm to (98.1, 78.1)
- moved R42 44.1 mm to (98.2, 81.5)
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Routing:
- net Net-(U1-PA12): track 0.00 -> 50.7 mm, vias 0 -> 4
- net Net-(U1-PA11): track 0.00 -> 50.2 mm, vias 0 -> 4
- net Net-(U1-PA2): track 0.00 -> 19.9 mm
- net Net-(U1-PA3): track 0.00 -> 17.9 mm
- net /UsbAndPower/USB_D+: track 2.20 -> 14.0 mm
- net /UsbAndPower/USB_D-: track 0.00 -> 10.5 mm
- net /DebugAndUart/TARGET_TXD: track 9.19 -> 16.5 mm, vias 0 -> 1
- net /DebugAndUart/TARGET_SWCLK: track 14.0 -> 8.23 mm
- net /DebugAndUart/TARGET_SWDIO: track 12.7 -> 7.61 mm
- net +3.3V: track 12.8 -> 16.9 mm
- net /DebugAndUart/TARGET_RXD: track 9.55 -> 12.7 mm
- net Net-(Q3-D): track 5.25 -> 2.38 mm
- net Net-(Q3-G): track 0.00 -> 2.83 mm
- net Net-(Q4-D): track 2.58 -> 0.00 mm
- net Net-(U1-PB14): track 10.1 -> 8.44 mm
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