File: DapLink_STM32F103CBT6.kicad_pcb (KiCad board)
At the start: 2 copper layers, 154 x 97.5 mm, 103 parts, among them J1 Conn_01x03_Pin, J2 Conn_01x03_Pin, J3 Conn_01x08_Pin, J4 USB_C_Receptacle_USB2.0_16P, J5 Conn_01x08_Pin, J6 Conn_01x08_Pin, J7 Conn_01x03_Pin, Q1 SI2306, Q2 SI2306, Q3 SI2306, Q4 SI2301, Q5 SI2306, Q6 SI2306, Q7 SI2306, Q8 SI2306, SW1 SKQGAFE010, U1 STM32F103CBTx, U2 LM1117MP-3.3, U3 RT9193-18GB, U4 RT9193-33GB, U5 HT75xx-1-SOT89, U6 TXB0104PW, Y1 Crystal_GND24

Commit message: temp
Parts:
- moved C12 45.0 mm to (48.0, 73.6), turned to 90 degrees
- moved U2 41.5 mm to (53.7, 71.7), turned to 0 degrees
- moved C20 39.3 mm to (45.2, 81.8), turned to -90 degrees
- moved U5 34.6 mm to (43.7, 77.6), turned to -90 degrees
- moved C15 31.2 mm to (55.0, 64.6), turned to 180 degrees
- moved C21 30.8 mm to (43.2, 73.3), turned to 0 degrees
- moved FB1 7.40 mm to (48.5, 86.9), turned to 0 degrees
- moved C10 7.36 mm to (59.6, 60.2)
- moved R21 7.36 mm to (59.7, 56.2)
- moved R26 1.48 mm to (43.1, 81.8), turned to -90 degrees
- moved C16 1.29 mm to (58.3, 80.6)
- moved C18 1.29 mm to (55.8, 77.3)
- moved U3 1.29 mm to (55.2, 80.9)
- moved C13 1.29 mm to (55.8, 84.5)
- moved C19 1.13 mm to (49.5, 77.3)
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Routing:
- net +3.3V: track 16.9 -> 47.1 mm
- net +5V: track 11.2 -> 34.9 mm
- net /UsbAndPower/USB_VBUS: track 1.88 -> 15.9 mm, vias 1 -> 2
- net GND: track 63.8 -> 64.8 mm, vias 7 -> 13
- net Net-(J4-CC2): track 11.8 -> 11.3 mm

Commit message: temp
Parts:
- moved J1 50.5 mm to (71.7, 116.7)
- moved R7 50.5 mm to (59.6, 118.0)
- moved R9 50.5 mm to (68.4, 119.4)
- moved J2 50.5 mm to (63.9, 116.6)
- moved R3 26.1 mm to (83.4, 106.8)
- moved D3 26.1 mm to (83.4, 110.8)
- moved R2 25.1 mm to (81.4, 106.8)
- moved D2 25.1 mm to (81.4, 110.8)
- moved R1 24.1 mm to (79.4, 106.8)
- moved D1 24.1 mm to (79.4, 110.8)
- moved J3 18.5 mm to (79.6, 69.8)
- moved C10 18.3 mm to (61.8, 78.4)
- moved R21 18.3 mm to (61.8, 74.4)
- moved Q1 18.1 mm to (73.3, 78.2)
- moved R20 18.1 mm to (70.6, 78.4)
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Routing:
- net +3.3V: track 47.1 -> 134.4 mm, vias 0 -> 14
- net /Mcu/IF_RXD: track 0.00 -> 30.5 mm, vias 0 -> 5
- net /Mcu/IF_RESET: track 1.92 -> 30.1 mm, vias 1 -> 4
- net /Mcu/IF_TXD: track 0.00 -> 27.2 mm, vias 0 -> 2
- net /Mcu/IF_SWDIO: track 0.00 -> 21.9 mm, vias 0 -> 2
- net Net-(D7-A): track 0.00 -> 2.80 mm
- net Net-(D6-A): track 0.00 -> 2.77 mm
- net Net-(Q1-G): track 0.00 -> 1.84 mm
- net Net-(Q2-G): track 0.00 -> 1.84 mm
- net Net-(D7-K): track 0.00 -> 1.79 mm
- net Net-(D6-K): track 0.00 -> 1.79 mm
- net GND: vias 13 -> 15

Commit message: temp
Parts:
- moved R18 21.4 mm to (64.1, 95.6), turned to 90 degrees
- moved R19 20.1 mm to (64.1, 99.3), turned to 90 degrees
- moved J7 8.30 mm to (98.1, 69.8)
- moved R41 8.30 mm to (93.0, 73.2)
- moved R42 8.30 mm to (98.2, 73.2)
- moved Q1 4.69 mm to (77.0, 75.3)
- moved SW1 3.81 mm to (55.6, 97.7)
- moved Q2 3.34 mm to (69.4, 75.3)
- moved C1 3.28 mm to (62.0, 99.3)
- moved R4 3.26 mm to (62.0, 95.6)
- moved R20 2.61 mm to (73.2, 78.2), turned to 0 degrees
- moved R5 2.22 mm to (80.4, 82.5)
- moved R6 2.22 mm to (82.4, 82.5)
- moved D4 2.22 mm to (80.4, 86.3)
- moved D5 2.22 mm to (82.4, 86.3)
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Routing:
- net /UsbAndPower/USB_CONNECT: track 2.17 -> 58.7 mm, vias 0 -> 4
- net +1.8V_LDO: track 2.49 -> 50.1 mm, vias 0 -> 4
- net /DebugAndUart/TARGET_RESET: track 0.00 -> 34.3 mm, vias 0 -> 4
- net /Mcu/IF_SWO: track 0.00 -> 28.5 mm, vias 0 -> 3
- net Net-(U1-PB0): track 0.00 -> 16.8 mm, vias 0 -> 2
- net /Mcu/IF_SWCLK: track 0.00 -> 15.8 mm, vias 0 -> 1
- net Net-(U1-PA0): track 0.00 -> 13.3 mm, vias 0 -> 2
- net /Mcu/LED_CONNECTED: track 0.00 -> 11.6 mm
- net +3.3V: track 134.4 -> 123.0 mm, vias 14 -> 16
- net /Mcu/IF_RESET: track 30.1 -> 25.6 mm, vias 4 -> 3
- net Net-(D7-K): track 1.79 -> 3.49 mm
- net Net-(D6-K): track 1.79 -> 3.49 mm
- net /Mcu/IF_SWDIO: track 21.9 -> 23.3 mm, vias 2 -> 1
- net Net-(U1-PA12): track 50.7 -> 51.8 mm
- net /Mcu/IF_TXD: track 27.2 -> 28.2 mm, vias 2 -> 3
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
Commit message: temp
Parts:
- moved R9 19.1 mm to (72.3, 100.7), turned to 0 degrees
- moved R8 13.5 mm to (69.3, 100.6), turned to -90 degrees
- moved R7 11.0 mm to (57.1, 107.3), turned to -90 degrees
- moved J1 9.51 mm to (69.2, 107.5), turned to 90 degrees
- moved J2 9.25 mm to (65.6, 107.5), turned to -90 degrees
- moved D1 7.70 mm to (86.6, 108.1), turned to 0 degrees
- moved D3 7.43 mm to (86.6, 104.1), turned to 0 degrees
- moved D2 7.02 mm to (86.6, 106.1), turned to 0 degrees
- moved R1 3.47 mm to (82.6, 108.1), turned to 0 degrees
- moved R3 2.81 mm to (82.6, 104.1), turned to 0 degrees
- moved R2 1.40 mm to (82.6, 106.1), turned to 0 degrees
Routing:
- net /Mcu/LED_nHID: track 0.00 -> 26.0 mm, vias 0 -> 2
- net /Mcu/LED_nCDC: track 0.00 -> 23.5 mm, vias 0 -> 2
- net /Mcu/LED_nMSC: track 0.00 -> 22.0 mm, vias 0 -> 2
- net Net-(U1-PB0): track 16.8 -> 4.89 mm
- net /DebugAndUart/TARGET_RESET: track 34.3 -> 31.6 mm, vias 4 -> 2
- net /UsbAndPower/USB_CONNECT: track 58.7 -> 57.5 mm

Commit message: temp gnd
Parts:
- moved J2 7.60 mm to (58.0, 107.7)
- moved J1 4.14 mm to (65.1, 107.7)
- moved R7 2.69 mm to (56.4, 104.7), turned to 180 degrees
- moved R8 2.11 mm to (69.1, 98.5), turned to 180 degrees
- moved R9 1.30 mm to (73.0, 99.6), turned to 180 degrees
- moved R42 1.20 mm to (98.3, 74.4)
- moved J7 1.20 mm to (98.2, 71.0)
- moved R41 1.20 mm to (93.1, 74.4)
- moved SW1 0.78 mm to (56.2, 98.2)
- moved C9 0.30 mm to (63.7, 86.3)
- moved C6 0.20 mm to (64.3, 84.1)
Routing:
- net GND: track 64.4 -> 405.7 mm, vias 15 -> 220
- net +3.3V: track 123.0 -> 218.5 mm, vias 16 -> 32
- net +1.8V: track 10.6 -> 41.0 mm, vias 2 -> 5
- net Net-(U1-BOOT0): track 0.00 -> 30.4 mm, vias 0 -> 4
- net /Mcu/LED_RUNNING: track 0.00 -> 17.1 mm, vias 0 -> 2
- net +1.8V_Target: track 0.00 -> 14.2 mm, vias 0 -> 2
- net /Mcu/BOOT1: track 0.00 -> 13.6 mm, vias 0 -> 1
- net /UsbAndPower/USB_D+: track 14.0 -> 23.8 mm, vias 0 -> 2
- net Net-(U1-PB2): track 0.00 -> 9.37 mm, vias 0 -> 2
- net /DebugAndUart/TARGET_RESET: track 31.6 -> 39.1 mm, vias 2 -> 0
- net /DebugAndUart/TARGET_1v8_RESET: track 0.00 -> 7.53 mm
- net /DebugAndUart/TARGET_SWCLK: track 8.23 -> 14.0 mm
- net /DebugAndUart/TARGET_SWDIO: track 7.61 -> 12.6 mm
- net +1.8V_LDO: track 50.1 -> 54.9 mm
- net /Mcu/BOOT0: track 0.00 -> 3.01 mm
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
Commit message: temp
Parts:
- moved H2 365.4 mm to (40.5, 109.0)
- moved H4 301.7 mm to (103.0, 109.0)
- moved H3 289.9 mm to (103.0, 68.5)
- moved H1 214.9 mm to (40.5, 68.5)
- moved R41 3.20 mm to (89.9, 74.4)
- moved R42 3.20 mm to (95.1, 74.4)
- moved J7 3.20 mm to (95.0, 71.0)
Routing:
- net GND: track 405.7 -> 673.9 mm, vias 220 -> 219
- net +1.8V_Target: track 14.2 -> 16.7 mm
- net +1.8V: track 41.0 -> 43.0 mm
- net +1.8V_LDO: track 54.9 -> 53.7 mm
- net /Mcu/IF_RESET: track 25.6 -> 26.6 mm
Other:
- board size 154 x 97.5 mm -> 72.5 x 49.5 mm

Commit message: drc ok
Routing:
- net GND: track 673.9 -> 682.8 mm
Changed lines of the file:
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@@
 	)
 	(gr_rect
-		(start 35 64)
-		(end 107.5 113.5)
+		(start 36 64)
+		(end 108.5 113.5)
 		(stroke
 			(width 0.2)
@@
 	)
 	(segment
+		(start 63.68462 90.55962)
+		(end 63.68462 88.21538)
+		(width 0.3)
+		(layer "B.Cu")
+		(net 2)
+	)
+	(segment
 		(start 96.7 96.4)
 		(end 96.7 98)
@@
 	)
 	(segment
+		(start 57.8 102.7)
+		(end 58.5 102.7)
+		(width 0.3)
+		(layer "B.Cu")
+		(net 2)
+	)
+	(segment
 		(start 66.7 84.9)
 		(end 67.4 84.2)
@@
 	)
 	(segment
+		(start 63.68462 88.21538)
+		(end 63.8 88.1)
+		(width 0.3)
+		(layer "B.Cu")
+		(net 2)
+	)
+	(segment
 		(start 68.4 78.1)
 		(end 69.5 79.2)
@@
 	)
 	(segment
+		(start 58.5 102.7)
+		(end 59.4 103.6)
+		(width 0.3)
+		(layer "B.Cu")
+		(net 2)
+	)
+	(segment
 		(start 99.5 104.3)
 		(end 99.5 102)
@@
 	)
 	(segment
+		(start 59.2 103.8)
+		(end 59.2 105.1)
+		(width 0.3)
+		(layer "B.Cu")
+		(net 2)
+	)
+	(segment
 		(start 89 99.1)
 		(end 89 102.5)
@@
 	)
 	(segment
+		(start 53.8 104.8)
+		(end 53.8 101.9)
+		(width 0.3)
+		(layer "B.Cu")
+		(net 2)
+	)
+	(segment
 		(start 65.8 97.8)
 		(end 65.8 98.7)
@@
 	)
 	(segment
+		(start 59.4 103.6)
+		(end 59.2 103.8)
+		(width 0.3)
+		(layer "B.Cu")
+		(net 2)
+	)
+	(segment
 		(start 62.21875 87.85)
 		(end 63.61875 89.25)
@@
 	)
 	(segment
-		(start 84 88.9)
-		(end 83.7125 89.1875)
-		(width 0.6)
-		(layer "F.Cu")
-		(net 69)
-	)
-	(segment
 		(start 93.4 98.5)
 		(end 93.4 99.5)
@@
 	)
 	(segment
-		(start 83.7125 89.1875)
-		(end 83.7125 90.2)
-		(width 0.6)
-		(layer "F.Cu")
-		(net 69)
-	)
-	(segment
 		(start 88.765 95.5)
 		(end 86.5 97.765)
@@
 	)
 	(segment
+		(start 83.9 88.9)
+		(end 83.7125 89.0875)
+		(width 0.6)
+		(layer "F.Cu")
+		(net 69)
+	)
+	(segment
 		(start 89.8875 96.6875)
 		(end 90.6 97.4)
@@
 	)
 	(segment
+		(start 83.7125 89.0875)
+		(end 83.7125 90.2)
+		(width 0.6)
+		(layer "F.Cu")
+		(net 69)
+	)
+	(segment
 		(start 90.6 97.4)
 		(end 92.3 97.4)
@@
 	)
 	(via
-		(at 84 88.9)
+		(at 83.9 88.9)
 		(size 0.6)
 		(drill 0.3)
@@
 	)
 	(segment
-		(start 86.165 98.1)
-		(end 86.5 97.765)
+		(start 84.429291 97.9)
+		(end 86.365 97.9)
 		(width 0.3)
 		(layer "B.Cu")
@@
 	)
 	(segment
-		(start 84 97.4)
-		(end 84.7 98.1)
+		(start 86.365 97.9)
+		(end 86.5 97.765)
 		(width 0.3)
 		(layer "B.Cu")
@@
 	)
 	(segment
-		(start 84.7 98.1)
-		(end 86.165 98.1)
+		(start 83.9 88.9)
+		(end 83.9 97.370709)
 		(width 0.3)
 		(layer "B.Cu")
@@
 	)
 	(segment
-		(start 84 88.9)
-		(end 84 97.4)
+		(start 83.9 97.370709)
+		(end 84.429291 97.9)
 		(width 0.3)
 		(layer "B.Cu")

Commit message: before rename led
Parts:
- moved D1 6.23 mm to (80.4, 108.3)
- moved D2 6.23 mm to (80.4, 106.3)
- moved D3 6.23 mm to (80.4, 104.3)
- moved R1 6.23 mm to (76.4, 108.3)
- moved R2 6.23 mm to (76.4, 106.3)
- moved R3 6.23 mm to (76.4, 104.3)
- moved D4 5.31 mm to (80.1, 81.0), turned to -90 degrees
- moved D5 5.30 mm to (82.2, 81.0), turned to -90 degrees
- moved R5 3.98 mm to (76.5, 81.7), turned to 180 degrees
- moved R6 2.31 mm to (82.2, 84.8), turned to -90 degrees
Routing:
- net GND: track 682.8 -> 16.5 mm, vias 219 -> 310
- net /Mcu/LED_nMSC: track 22.1 -> 15.9 mm
- net /Mcu/LED_nHID: track 26.1 -> 20.4 mm
- net /Mcu/LED_nCDC: track 23.8 -> 18.1 mm
- net /Mcu/LED_RUNNING: track 17.1 -> 11.8 mm
- net /Mcu/LED_CONNECTED: track 11.4 -> 6.56 mm
- net +3.3V: track 218.4 -> 221.2 mm
- net Net-(U1-PB2): track 9.37 -> 7.39 mm
- net +1.8V_LDO: track 53.7 -> 52.3 mm
- net Net-(U1-PA0): track 13.3 -> 12.3 mm
- net Net-(D4-A): track 1.95 -> 2.79 mm
- net Net-(J4-CC1): track 9.53 -> 9.00 mm
- added copper zone on B.Cu, net GND
- added copper zone on F.Cu, net GND
