File: DapLink_STM32F103CBT6.kicad_pcb (KiCad board)
At the start: 2 copper layers, 72.5 x 49.5 mm, 103 parts, among them J1 Conn_01x03_Pin, J2 Conn_01x03_Pin, J3 Conn_01x08_Pin, J4 USB_C_Receptacle_USB2.0_16P, J5 Conn_01x08_Pin, J6 Conn_01x08_Pin, J7 Conn_01x03_Pin, Q1 SI2306, Q2 SI2306, Q3 SI2306, Q4 SI2301, Q5 SI2306, Q6 SI2306, Q7 SI2306, Q8 SI2306, SW1 SKQGAFE010, U1 STM32F103CBTx, U2 LM1117MP-3.3, U3 RT9193-18GB, U4 RT9193-33GB, U5 HT75xx-1-SOT89, U6 TXB0104PW, Y1 Crystal_GND24

Commit message: looks good v1
Routing:
- net GND: vias 310 -> 315
Other:
- board text added: "1.8V GND 1V8_SWCLK 1V8_SWDIO 1V8_TXD 1V8_RXD 1V8_SWO 1V8_RESET"
- board text added: "3.3V BOOT1 GND"
- board text added: "3.3V GND IF_SWCLK IF_SWDIO IF_TXD IF_RXD IF_SWO IF_RESET"
- board text added: "3.3V GND SWCLK SWDIO TXD RXD SWO RESET"
- board text added: "DAPLINK roger225"
- board text added: "GND BOOT0 3.3V"
- board text added: "H Boot0 L"
- board text added: "L Boot1 H"
- board text added: "LDO 1.8V TARGET"
